File: sweet-p.kicad_sch (KiCad schematic)
At the start: 11 parts, among them J1 RJ45, J2 Conn_01x04_Female, J3 Screw_Terminal_01x03, J4 Screw_Terminal_01x03, J5 Screw_Terminal_01x02, J6 Screw_Terminal_01x03, U1 RFM95W-868S2, U2 SAM-M8Q

Commit message: update
Parts:
- removed A1: Adafruit_Feather_M0_RFM9x_LoRa_Radio, Module:Adafruit_Feather_M0_RFM, symbol MCU_Module:Adafruit_Feather_M0_RFM9x_LoRa_Radio
- removed BT1: Battery, Battery:BatteryHolder_Keystone_2479_3xAAA, symbol Device:Battery
- removed J1: RJ45, Connector_RJ:RJ45_Amphenol_54602-x08_Horizontal, symbol Connector:RJ45
- removed J4, J6: Screw_Terminal_01x03, TerminalBlock_Phoenix:TerminalBlock_Phoenix_PT-1,5-3-5.0-H_1x03_P5.00mm_Horizontal, symbol Connector:Screw_Terminal_01x03
- removed U2: SAM-M8Q, RF_GPS:ublox_SAM-M8Q, symbol RF_GPS:SAM-M8Q
- added A1: Adafruit_Feather_Generic, Module:Adafruit_Feather, symbol MCU_Module:Adafruit_Feather_Generic
- added H1, H2: MountingHole, MountingHole:MountingHole_3.2mm_M3, symbol Mechanical:MountingHole
- added J4: Screw_Terminal_01x04, TerminalBlock_Phoenix:TerminalBlock_Phoenix_PT-1,5-4-5.0-H_1x04_P5.00mm_Horizontal, symbol Connector:Screw_Terminal_01x04
- added J5: Conn_01x06_Female, Connector_PinSocket_2.54mm:PinSocket_1x06_P2.54mm_Vertical, symbol Connector:Conn_01x06_Female
- added J6: Conn_01x08_Female, Connector_PinSocket_2.54mm:PinSocket_1x08_P2.54mm_Vertical, symbol Connector:Conn_01x08_Female
- added U2: Adafruit-Mini-GPS, gps:adafruit_mini_gps, symbol sweet-p:Adafruit-Mini-GPS
- J2: renamed from J5; footprint TerminalBlock_Phoenix:TerminalBlock_Phoenix_MKDS-1,5-2_1x02_P5.00mm_Horizontal -> TerminalBlock_Phoenix:TerminalBlock_Phoenix_PT-1,5-2-5.0-H_1x02_P5.00mm_Horizontal
- renumbered J3 to J1, J2 to J3
Other:
- note added: "add power control to gps"
- note added: "add simple rtc"

Commit message: update
Parts:
- added H?: MountingHole, MountingHole:MountingHole_3.2mm_M3, symbol Mechanical:MountingHole
Changed lines of the file:
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@@
     (pin "6")
+  )
+  (symbol (lib_id "Mechanical:MountingHole") (at 96.52 142.24 0) (unit 1)
+    (in_bom yes) (on_board yes) (fields_autoplaced)
+    (property "Reference" "H?" (id 0) (at 99.06 140.9699 0)
+      (effects (font (size 1.27 1.27)) (justify left))
+    )
+    (property "Value" "MountingHole" (id 1) (at 99.06 143.5099 0)
+      (effects (font (size 1.27 1.27)) (justify left))
+    )
+    (property "Footprint" "MountingHole:MountingHole_3.2mm_M3" (id 2) (at 96.52 142.24 0)
+      (effects (font (size 1.27 1.27)) hide)
+    )
+    (property "Datasheet" "~" (id 3) (at 96.52 142.24 0)
+      (effects (font (size 1.27 1.27)) hide)
+    )
   )
   (symbol (lib_id "Mechanical:MountingHole") (at 86.36 121.92 0) (unit 1)
@@
       (reference "H2") (unit 1) (value "MountingHole") (footprint "MountingHole:MountingHole_3.2mm_M3")
     )
+    (path "/318e249e-412d-4076-86d9-3d57986e4360"
+      (reference "H?") (unit 1) (value "MountingHole") (footprint "MountingHole:MountingHole_3.2mm_M3")
+    )
     (path "/356a682b-39b5-417e-8373-9ae81bd97f29"

Commit message: update
Parts:
- removed J3: Conn_01x04_Female, footprints:ssd1306_b, symbol Connector:Conn_01x04_Female
- added BT1: CR1220, picoco2:CR1220-2, symbol Device:Battery
- added C1, C2: 10uF, Capacitor_SMD:C_0603_1608Metric_Pad1.08x0.95mm_HandSolder, symbol Device:C
- added J6: Conn_01x03_Female, Connector_PinSocket_2.54mm:PinSocket_1x03_P2.54mm_Vertical, symbol Connector:Conn_01x03_Female
- added J7: Micro_SD_Card, footprints:DM3D-SF_outline, symbol Connector:Micro_SD_Card
- added JP1, JP2: SolderJumper_2_Open, Jumper:SolderJumper-2_P1.3mm_Open_Pad1.0x1.5mm, symbol Jumper:SolderJumper_2_Open
- added Q1, Q2: Q_NMOS_GDS, Package_TO_SOT_SMD:SOT-23, symbol Device:Q_NMOS_GDS
- added R2, R3: 4.7K, Resistor_SMD:R_0603_1608Metric_Pad0.98x0.95mm_HandSolder, symbol Device:R
- added R5: 10K, Resistor_SMD:R_0603_1608Metric_Pad0.98x0.95mm_HandSolder, symbol Device:R
- added R6, R7: R, Resistor_SMD:R_0603_1608Metric_Pad0.98x0.95mm_HandSolder, symbol Device:R
- added R8: 1K, Resistor_SMD:R_0603_1608Metric_Pad0.98x0.95mm_HandSolder, symbol Device:R
- added R?: 10K, Resistor_THT:R_Axial_DIN0204_L3.6mm_D1.6mm_P7.62mm_Horizontal, symbol Device:R
- added SW?: SW_Push, Button_Switch_THT:SW_Tactile_SPST_Angled_PTS645Vx31-2LFS, symbol Switch:SW_Push
- added U2: ssd1306, footprints:ssd1306_a, symbol picoco2:ssd1306
- added U4: PCF8523T, Package_SO:SOIC-8_3.9x4.9mm_P1.27mm, symbol Timer_RTC:PCF8523T
- added Y1: 32KHz, Crystal:Crystal_SMD_Abracon_ABS25-4Pin_8.0x3.8mm, symbol Device:Crystal_GND23
- gave numbers to parts that had none: 1
- renumbered J6 to J8, U2 to U3
Connections:
- net GND_1: now reaches U3.1 (GND)
- net GND_1: now also JP2.2 (B), Q2.2 (D)
- new net: U4.2 (OSCO), Y1.1
- new net: U4.1 (OSCI), Y1.4
- new net: BT1.1 (+), U4.3 (VBAT)
- new net: C1.1, R8.1, U4.8 (VDD)
- new net: J6.2 (Pin_2), R5.1
- new net +3V3: C2.1, J7.4 (VDD), R2.1, R3.1, R8.2, R?.1, U2.2 (3V3)
- new net BUT_A: R?.2, SW?.1
- new net GND: BT1.2 (-), C1.2, C2.2, J7.6 (VSS), JP1.1 (A), JP2.1 (A), Q1.3 (S), Q2.3 (S), R5.2, R6.2, R7.2, SW?.2, U2.1 (GND), U4.4 (VSS)
- new net GND_1_EN: Q2.1 (G), R7.1
- new net GND_2: JP1.2 (B), Q1.2 (D)
- new net GND_2_EN: Q1.1 (G), R6.1
- new net MISO: J7.7 (DAT0)
- new net MOSI: J7.3 (CMD)
- new net RTC_INT: U4.7 (~{INT1}/CLKOUT)
- new net SCK: J7.5 (CLK)
- new net SCL: R3.2, U2.3 (SCL), U4.6 (SCL)
- new net SDA: R2.2, U2.4 (SDA), U4.5 (SDA)
- new net SD_CS: J7.2 (DAT3/CD)
- new net WRITE_EN: J6.3 (Pin_3)
Other:
- note added: "i2c pullups"
- note added: "write permit"
- note removed: "add power control to gps"
- moved on the sheet: A1, AE1, H1, H2, H3, J1, J2, J4, J5, J8, U1, U3

Commit message: update
Parts:
- added R1, R4: 4.7K, Resistor_THT:R_Axial_DIN0204_L3.6mm_D1.6mm_P7.62mm_Horizontal, symbol Device:R
- added R5: 1K, Resistor_SMD:R_0603_1608Metric_Pad0.98x0.95mm_HandSolder, symbol Device:R
- gave numbers to parts that had none: 2
- renumbered J4 to J3, J5 to J4, J6 to J5, J7 to J6, J8 to J7, R8 to R10, R5 to R7, R6 to R8, R7 to R9
Connections:
- net +3V3: now also R1.1, R4.1, R5.2
- net BUT_A: now also R5.1
- net SCL: now also R4.2
- net SDA: now also R1.2

Commit message: update
Parts:
- removed A1: Adafruit_Feather_Generic, Module:Adafruit_Feather, symbol MCU_Module:Adafruit_Feather_Generic
- removed BT1: CR1220, picoco2:CR1220-2, symbol Device:Battery
- removed C1, C2: 10uF, Capacitor_SMD:C_0603_1608Metric_Pad1.08x0.95mm_HandSolder, symbol Device:C
- removed R10: 1K, Resistor_SMD:R_0603_1608Metric_Pad0.98x0.95mm_HandSolder, symbol Device:R
- removed U4: PCF8523T, Package_SO:SOIC-8_3.9x4.9mm_P1.27mm, symbol Timer_RTC:PCF8523T
- removed Y1: 32KHz, Crystal:Crystal_SMD_Abracon_ABS25-4Pin_8.0x3.8mm, symbol Device:Crystal_GND23
- added A1: Adafruit_Feather_M0_Express, Module:Adafruit_Feather, symbol MCU_Module:Adafruit_Feather_M0_Express
- added H4: MountingHole, MountingHole:MountingHole_3.2mm_M3, symbol Mechanical:MountingHole
- added J2: Conn_01x03_Female, Connector_PinSocket_2.54mm:PinSocket_1x03_P2.54mm_Vertical, symbol Connector:Conn_01x03_Female
- added R1: 4.7K, Resistor_THT:R_Axial_DIN0204_L3.6mm_D1.6mm_P7.62mm_Horizontal, symbol Device:R
- added R13: 10K, Resistor_SMD:R_0603_1608Metric_Pad0.98x0.95mm_HandSolder, symbol Device:R
- added R14: R, Resistor_THT:R_Axial_DIN0204_L3.6mm_D1.6mm_P7.62mm_Horizontal, symbol Device:R
- added R2: 4.7K, Resistor_SMD:R_0603_1608Metric_Pad0.98x0.95mm_HandSolder, symbol Device:R
- added R9: 10K, Resistor_THT:R_Axial_DIN0204_L3.6mm_D1.6mm_P7.62mm_Horizontal, symbol Device:R
- added U4: ds3231, footprints:ds3231_adafruit_breakout, symbol adafruit_ds3231:ds3231
- renumbered J4 to J3, J7 to J4, J6 to J5, J2 to J6, J3 to J7, J5 to J8, JP2 to JP1, JP1 to JP2, Q2 to Q1, Q1 to Q2, R7 to R10, R8 to R11, R9 to R12, R1 to R3, R2 to R4, R3 to R5, R4 to R6, R5 to R7, R6 to R8
Connections:
- net +3V3: now also J1.1 (Pin_1), J7.2 (Pin_2), U1.13 (3.3V), U3.3 (VIN), A1.2 (3V3), R1.1, R13.1, R14.1, R2.1, U4.1 (VIN)
- net BUT_A: now also A1.5 (DAC0/A0)
- net GND: now also J1.3 (Pin_3), J6.2 (Pin_2), U1.1 (GND), U1.10 (GND), U1.8 (GND), A1.16 (GND), A1.4 (GND), J2.3 (Pin_3), R9.2, U4.2 (GND)
- net GND_1: now also U3.10 (GND)
- net GND_1_EN: now also A1.9 (A4)
- net GND_2: now also J7.1 (Pin_1)
- net GND_2_EN: now also A1.10 (A5)
- net MISO: now also U1.2 (MISO), A1.13 (MISO/D22)
- net MOSI: now also U1.3 (MOSI), A1.12 (MOSI/D23)
- net RTC_INT: now also A1.25 (D13), R13.2, R14.2, U4.7 (SQW)
- net SCK: now also U1.4 (SCK), A1.11 (SCK/D24)
- net SCL: now also U3.9 (SCL), A1.18 (SCL/D21), U4.3 (SCL)
- net SDA: now also U3.8 (SDA), A1.17 (SDA/D20), U4.4 (SDA)
- net SD_CS: now also A1.22 (D10)
- net VBAT: now also A1.28 (VBAT)
- net VBUS: now also J6.1 (Pin_1), A1.26 (USB)
- net WRITE_EN: now also A1.8 (A3)
- net ONEWIRE: now reaches J1.2 (Pin_2)
- net ONEWIRE: now also A1.19 (D5), R1.2, R2.2
- net GPS_RST: now reaches U3.7 (RST)
- net GPS_RST: now also A1.7 (A2)
- net at J8.2 (Pin_2), R10.1: now also R9.1
- net RX: now reaches J7.3 (Pin_3)
- net RX: now also A1.14 (RX/D0)
- net TX: now reaches J7.4 (Pin_4)
- net TX: now also A1.15 (TX/D1)
- net at AE1.2 (Shield): now also U1.9 (ANT)
- net LORA_CS: now reaches U1.5 (NSS)
- net LORA_CS: now also A1.20 (D6)
- net LORA_RST: now reaches U1.6 (RESET)
- net LORA_RST: now also A1.21 (D9)
- new net EN: A1.27 (EN), J2.2 (Pin_2)
- new net RX2: A1.23 (D11)
- new net SAT_EN: A1.6 (A1)
- new net TX2: A1.24 (D12)
Other:
- note added: "ext power"
- note added: "on/off"
- note removed: "add RX + TX + 3V + GND + 5V for UART application (ultrasonic, satellite)"
- note removed: "add simple rtc"
- moved on the sheet: AE1, H1, H2, H3, J1, J3, J4, J5, J6, J7

Commit message: laid out power
Connections:
- net +3V3: now also J3.4 (Pin_4)
- net GND: now also AE1.1 (A), J3.6 (Pin_6), J4.1 (Pin_1), J4.8 (Pin_8)
- net RX2: now also J3.2 (Pin_2)
- net SAT_EN: now also J4.6 (Pin_6)
- net TX2: now also J3.3 (Pin_3)
- net VBAT: now also J4.7 (Pin_7)
Other:
- moved on the sheet: AE1, J3, J4
