File: sweet-p.kicad_pcb (KiCad board)
At the start: 2 copper layers, 11 parts, among them J1 RJ45, J2 Conn_01x04_Female, J3 Screw_Terminal_01x03, J4 Screw_Terminal_01x03, J5 Screw_Terminal_01x02, J6 Screw_Terminal_01x03, U1 RFM95W-868S2, U2 SAM-M8Q

Commit message: update
Parts:
- removed BT1: Battery, Battery:BatteryHolder_Keystone_2479_3xAAA
- added H1: MountingHole, MountingHole:MountingHole_3.2mm_M3, F.Cu at (226.8, 121.0)
- added H2: MountingHole, MountingHole:MountingHole_3.2mm_M3, F.Cu at (166.4, 120.8)
- A1: value Adafruit_Feather_M0_RFM9x_LoRa_Radio -> Adafruit_Feather_Generic; footprint Module:Adafruit_Feather_M0_RFM -> Module:Adafruit_Feather
- J1: value RJ45 -> Screw_Terminal_01x03; footprint Connector_RJ:RJ45_Amphenol_54602-x08_Horizontal -> TerminalBlock_Phoenix:TerminalBlock_Phoenix_PT-1,5-3-5.0-H_1x03_P5.00mm_Horizontal
- J2: value Conn_01x04_Female -> Screw_Terminal_01x02; footprint footprints:ssd1306_b -> TerminalBlock_Phoenix:TerminalBlock_Phoenix_PT-1,5-2-5.0-H_1x02_P5.00mm_Horizontal
- J3: value Screw_Terminal_01x03 -> Conn_01x04_Female; footprint TerminalBlock_Phoenix:TerminalBlock_Phoenix_PT-1,5-3-5.0-H_1x03_P5.00mm_Horizontal -> footprints:ssd1306_b
- J4: value Screw_Terminal_01x03 -> Screw_Terminal_01x04; footprint TerminalBlock_Phoenix:TerminalBlock_Phoenix_PT-1,5-3-5.0-H_1x03_P5.00mm_Horizontal -> TerminalBlock_Phoenix:TerminalBlock_Phoenix_PT-1,5-4-5.0-H_1x04_P5.00mm_Horizontal
- J5: value Screw_Terminal_01x02 -> Conn_01x06_Female; footprint TerminalBlock_Phoenix:TerminalBlock_Phoenix_MKDS-1,5-2_1x02_P5.00mm_Horizontal -> Connector_PinSocket_2.54mm:PinSocket_1x06_P2.54mm_Vertical
- J6: value Screw_Terminal_01x03 -> Conn_01x08_Female; footprint TerminalBlock_Phoenix:TerminalBlock_Phoenix_PT-1,5-3-5.0-H_1x03_P5.00mm_Horizontal -> Connector_PinSocket_2.54mm:PinSocket_1x08_P2.54mm_Vertical
- U2: value SAM-M8Q -> Adafruit-Mini-GPS; footprint RF_GPS:ublox_SAM-M8Q -> gps:adafruit_mini_gps
- moved J1 117.6 mm to (187.3, 116.0)
- moved A1 98.7 mm to (177.6, 108.4), turned to 90 degrees
- moved U2 87.3 mm to (216.4, 61.9)
- moved J2 73.3 mm to (174.4, 116.0)
- moved J4 40.7 mm to (204.6, 116.0)
- moved J6 38.2 mm to (227.7, 77.1), turned to 180 degrees
- moved J5 37.2 mm to (227.8, 84.3)
- moved U1 33.9 mm to (177.6, 76.6), turned to 180 degrees
- moved AE1 30.8 mm to (168.9, 62.9)
- moved J3 14.1 mm to (181.1, 61.4), turned to 90 degrees
Connections:
- U2 pad 1: Net-(U2-Pad1) -> unconnected-(U2-Pad1)
- U2 pad 10: Net-(U2-Pad1) -> unconnected-(U2-Pad10)
- U2 pad 11: Net-(U2-Pad1) -> unconnected-(U2-Pad11)
- U2 pad 4: Net-(U2-Pad1) -> unconnected-(U2-Pad4)
- U2 pad 5: Net-(U2-Pad1) -> unconnected-(U2-Pad5)
- U2 pad 6: Net-(U2-Pad1) -> unconnected-(U2-Pad6)
Other:
- board outline added: 68.1 x 69 mm

Commit message: update
Parts:
- added H3: MountingHole, MountingHole:MountingHole_3.2mm_M3, F.Cu at (167.0, 61.1)
- moved AE1 15.0 mm to (168.6, 77.9), turned to 90 degrees
- moved U1 6.87 mm to (182.7, 72.0), turned to -90 degrees
- moved J3 2.20 mm to (181.0, 59.2)
- moved J1 2.20 mm to (187.2, 113.8)
- moved J4 2.20 mm to (204.5, 113.8)
- moved J2 2.20 mm to (174.3, 113.8)
- moved A1 1.95 mm to (177.7, 106.5)
- moved U2 1.87 mm to (216.6, 60.0)
- moved H1 1.32 mm to (227.0, 119.7)
- moved H2 1.32 mm to (166.6, 119.5)
Other:
- board size 68.1 x 69 mm -> 68.1 x 66.8 mm

Commit message: update
Parts:
- added C1: 10uF, Capacitor_SMD:C_0603_1608Metric_Pad1.08x0.95mm_HandSolder, F.Cu at (45.9, 15.8)
- added C2: 10uF, Capacitor_SMD:C_0603_1608Metric_Pad1.08x0.95mm_HandSolder, F.Cu at (40.2, 12.2)
- added J7: Conn_01x08_Female, Connector_PinSocket_2.54mm:PinSocket_1x08_P2.54mm_Vertical, F.Cu at (68.0, 9.00)
- added JP1: SolderJumper_2_Open, Jumper:SolderJumper-2_P1.3mm_Open_Pad1.0x1.5mm, F.Cu at (50.6, 14.1)
- added JP2: SolderJumper_2_Open, Jumper:SolderJumper-2_P1.3mm_Open_Pad1.0x1.5mm, F.Cu at (57.6, 14.2)
- added Q1: Q_NMOS_GDS, Package_TO_SOT_SMD:SOT-23, F.Cu at (58.0, 8.20)
- added Q2: Q_NMOS_GDS, Package_TO_SOT_SMD:SOT-23, F.Cu at (51.1, 8.40)
- added R1: 4.7K, Resistor_SMD:R_0603_1608Metric_Pad0.98x0.95mm_HandSolder, F.Cu at (47.4, 20.4)
- added R2: 4.7K, Resistor_SMD:R_0603_1608Metric_Pad0.98x0.95mm_HandSolder, F.Cu at (40.3, 16.0)
- added R3: 10K, Resistor_THT:R_Axial_DIN0204_L3.6mm_D1.6mm_P7.62mm_Horizontal, F.Cu at (45.4, 12.4)
- added R4: 10K, Resistor_SMD:R_0603_1608Metric_Pad0.98x0.95mm_HandSolder, F.Cu at (34.2, 21.4)
- added R5: R, Resistor_SMD:R_0603_1608Metric_Pad0.98x0.95mm_HandSolder, F.Cu at (36.5, 10.7)
- added R6: R, Resistor_SMD:R_0603_1608Metric_Pad0.98x0.95mm_HandSolder, F.Cu at (45.0, 8.80)
- added R7: 1K, Resistor_SMD:R_0603_1608Metric_Pad0.98x0.95mm_HandSolder, F.Cu at (40.1, 8.60)
- added SW1: SW_Push, Button_Switch_THT:SW_Tactile_SPST_Angled_PTS645Vx31-2LFS, F.Cu at (5.11, 49.3)
- added U3: Adafruit-Mini-GPS, gps:adafruit_mini_gps, F.Cu at (55.4, 30.3)
- added U4: PCF8523T, Package_SO:SOIC-8_3.9x4.9mm_P1.27mm, F.Cu at (30.1, 12.3)
- added Y1: 32KHz, Crystal:Crystal_SMD_Abracon_ABS25-4Pin_8.0x3.8mm, F.Cu at (22.1, 12.3)
- J3: value Conn_01x04_Female -> Screw_Terminal_01x04; footprint footprints:ssd1306_b -> TerminalBlock_Phoenix:TerminalBlock_Phoenix_PT-1,5-4-5.0-H_1x04_P5.00mm_Horizontal
- J4: value Screw_Terminal_01x04 -> Conn_01x06_Female; footprint TerminalBlock_Phoenix:TerminalBlock_Phoenix_PT-1,5-4-5.0-H_1x04_P5.00mm_Horizontal -> Connector_PinSocket_2.54mm:PinSocket_1x06_P2.54mm_Vertical
- J5: value Conn_01x06_Female -> Conn_01x03_Female; footprint Connector_PinSocket_2.54mm:PinSocket_1x06_P2.54mm_Vertical -> Connector_PinSocket_2.54mm:PinSocket_1x03_P2.54mm_Vertical
- J6: value Conn_01x08_Female -> Micro_SD_Card; footprint Connector_PinSocket_2.54mm:PinSocket_1x08_P2.54mm_Vertical -> footprints:DM3D-SF_outline
- U2: value Adafruit-Mini-GPS -> ssd1306; footprint gps:adafruit_mini_gps -> footprints:ssd1306_a
- moved J6 230.6 mm to (5.20, 16.4), turned to -90 degrees
- moved J5 227.8 mm to (2.02, 54.3)
- moved U2 196.4 mm to (22.6, 29.3), turned to -90 degrees
- moved A1 180.4 mm to (16.8, 25.0)
- moved H3 173.2 mm to (3.70, 3.50)
- moved H2 171.4 mm to (3.70, 66.1)
- moved J1 169.9 mm to (25.5, 61.8)
- moved J2 169.8 mm to (12.7, 61.6)
- moved H1 169.8 mm to (66.0, 65.8)
- moved AE1 166.3 mm to (7.60, 36.2)
- moved U1 163.6 mm to (22.0, 41.4)
- moved J4 159.0 mm to (67.0, 33.9)
- moved J3 138.3 mm to (42.8, 62.0), turned to 0 degrees
Connections:
- J5 pad 2: unconnected-(J5-Pad2) -> Net-(J5-Pad2)
- J5 pad 3: unconnected-(J5-Pad3) -> WRITE_EN
- J6 pad 2: unconnected-(J6-Pad2) -> SD_CS
- J6 pad 3: unconnected-(J6-Pad3) -> MOSI
- J6 pad 4: unconnected-(J6-Pad4) -> +3V3
- J6 pad 5: unconnected-(J6-Pad5) -> SCK
- J6 pad 6: unconnected-(J6-Pad6) -> GND
- J6 pad 7: unconnected-(J6-Pad7) -> MISO
- U2 pad 1: unconnected-(U2-Pad1) -> GND
- U2 pad 2: unconnected-(U2-Pad2) -> +3V3
- U2 pad 3: unconnected-(U2-Pad3) -> SCL
- U2 pad 4: unconnected-(U2-Pad4) -> SDA
Other:
- board size 68.1 x 66.8 mm -> 70 x 70 mm

Commit message: update
Parts:
- added R10: 1K, Resistor_SMD:R_0603_1608Metric_Pad0.98x0.95mm_HandSolder, F.Cu at (33.4, 18.6)
- added R8: R, Resistor_SMD:R_0603_1608Metric_Pad0.98x0.95mm_HandSolder, F.Cu at (55.4, 20.8)
- added R9: R, Resistor_SMD:R_0603_1608Metric_Pad0.98x0.95mm_HandSolder, F.Cu at (49.6, 20.0)
- R1: footprint Resistor_SMD:R_0603_1608Metric_Pad0.98x0.95mm_HandSolder -> Resistor_THT:R_Axial_DIN0204_L3.6mm_D1.6mm_P7.62mm_Horizontal
- R3: value 10K -> 4.7K; footprint Resistor_THT:R_Axial_DIN0204_L3.6mm_D1.6mm_P7.62mm_Horizontal -> Resistor_SMD:R_0603_1608Metric_Pad0.98x0.95mm_HandSolder
- R4: value 10K -> 4.7K; footprint Resistor_SMD:R_0603_1608Metric_Pad0.98x0.95mm_HandSolder -> Resistor_THT:R_Axial_DIN0204_L3.6mm_D1.6mm_P7.62mm_Horizontal
- R5: value R -> 1K
- R6: value R -> 10K; footprint Resistor_SMD:R_0603_1608Metric_Pad0.98x0.95mm_HandSolder -> Resistor_THT:R_Axial_DIN0204_L3.6mm_D1.6mm_P7.62mm_Horizontal
- R7: value 1K -> 10K
- moved SW1 15.5 mm to (3.56, 33.9)
- moved R4 12.0 mm to (22.2, 20.6)
- moved R1 10.4 mm to (37.0, 20.8)
- moved AE1 8.80 mm to (4.40, 44.4), turned to 180 degrees
- moved R5 3.36 mm to (35.2, 13.8), turned to 90 degrees
- moved C2 1.86 mm to (39.1, 13.7)
- moved JP1 1.86 mm to (49.5, 15.6)
- moved JP2 1.86 mm to (56.5, 15.7)
- moved Q1 1.86 mm to (56.9, 9.70)
- moved Q2 1.86 mm to (50.0, 9.90)
- moved R2 1.86 mm to (39.2, 17.5)
- moved R3 1.86 mm to (44.3, 13.9)
- moved R6 1.86 mm to (43.9, 10.3)
- moved R7 1.86 mm to (39.0, 10.1)
- moved C1 1.86 mm to (44.8, 17.3)
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Connections:
- R2 pad 2: SCL -> SDA
- R3 pad 2: BUT_A -> SCL
- R4 pad 1: Net-(J5-Pad2) -> +3V3
- R4 pad 2: GND -> SCL
- R5 pad 1: GND_2_EN -> BUT_A
- R5 pad 2: GND -> +3V3
- R6 pad 1: GND_1_EN -> +3V3
- R6 pad 2: GND -> BUT_A
- R7 pad 1: Net-(C1-Pad1) -> Net-(J5-Pad2)
- R7 pad 2: +3V3 -> GND

Commit message: update
Parts:
- removed C1, C2: 10uF, Capacitor_SMD:C_0603_1608Metric_Pad1.08x0.95mm_HandSolder
- removed Y1: 32KHz, Crystal:Crystal_SMD_Abracon_ABS25-4Pin_8.0x3.8mm
- added H4: MountingHole, MountingHole:MountingHole_3.2mm_M3, F.Cu at (66.6, 3.40)
- added J8: Conn_01x03_Female, Connector_PinSocket_2.54mm:PinSocket_1x03_P2.54mm_Vertical, F.Cu at (17.0, 2.58)
- added R11: R, Resistor_SMD:R_0603_1608Metric_Pad0.98x0.95mm_HandSolder, F.Cu at (43.8, 21.8)
- added R12: R, Resistor_SMD:R_0603_1608Metric_Pad0.98x0.95mm_HandSolder, F.Cu at (28.9, 21.6)
- added R13: 10K, Resistor_SMD:R_0603_1608Metric_Pad0.98x0.95mm_HandSolder, F.Cu at (43.6, 42.7)
- added R14: R, Resistor_THT:R_Axial_DIN0204_L3.6mm_D1.6mm_P7.62mm_Horizontal, F.Cu at (43.6, 39.0)
- A1: value Adafruit_Feather_Generic -> Adafruit_Feather_M0_Express
- J2: value Screw_Terminal_01x02 -> Conn_01x03_Female; footprint TerminalBlock_Phoenix:TerminalBlock_Phoenix_PT-1,5-2-5.0-H_1x02_P5.00mm_Horizontal -> Connector_PinSocket_2.54mm:PinSocket_1x03_P2.54mm_Vertical
- J3: value Screw_Terminal_01x04 -> Conn_01x06_Female; footprint TerminalBlock_Phoenix:TerminalBlock_Phoenix_PT-1,5-4-5.0-H_1x04_P5.00mm_Horizontal -> Connector_PinSocket_2.54mm:PinSocket_1x06_P2.54mm_Vertical
- J4: value Conn_01x06_Female -> Conn_01x08_Female; footprint Connector_PinSocket_2.54mm:PinSocket_1x06_P2.54mm_Vertical -> Connector_PinSocket_2.54mm:PinSocket_1x08_P2.54mm_Vertical
- J5: value Conn_01x03_Female -> Micro_SD_Card; footprint Connector_PinSocket_2.54mm:PinSocket_1x03_P2.54mm_Vertical -> footprints:DM3D-SF_outline
- J6: value Micro_SD_Card -> Screw_Terminal_01x02; footprint footprints:DM3D-SF_outline -> TerminalBlock_Phoenix:TerminalBlock_Phoenix_PT-1,5-2-5.0-H_1x02_P5.00mm_Horizontal
- J7: value Conn_01x08_Female -> Screw_Terminal_01x04; footprint Connector_PinSocket_2.54mm:PinSocket_1x08_P2.54mm_Vertical -> TerminalBlock_Phoenix:TerminalBlock_Phoenix_PT-1,5-4-5.0-H_1x04_P5.00mm_Horizontal
- R10: value 1K -> 10K
- R3: footprint Resistor_SMD:R_0603_1608Metric_Pad0.98x0.95mm_HandSolder -> Resistor_THT:R_Axial_DIN0204_L3.6mm_D1.6mm_P7.62mm_Horizontal
- R4: footprint Resistor_THT:R_Axial_DIN0204_L3.6mm_D1.6mm_P7.62mm_Horizontal -> Resistor_SMD:R_0603_1608Metric_Pad0.98x0.95mm_HandSolder
- R5: value 1K -> 4.7K
- R6: value 10K -> 4.7K
- R7: value 10K -> 1K
- R8, R9: value R -> 10K; footprint Resistor_SMD:R_0603_1608Metric_Pad0.98x0.95mm_HandSolder -> Resistor_THT:R_Axial_DIN0204_L3.6mm_D1.6mm_P7.62mm_Horizontal
- U4: value PCF8523T -> ds3231; footprint Package_SO:SOIC-8_3.9x4.9mm_P1.27mm -> footprints:ds3231_adafruit_breakout; moved to B.Cu
- moved J2 70.0 mm to (50.2, 2.50), turned to 90 degrees
- moved J7 69.1 mm to (24.7, 62.9)
- moved J3 54.6 mm to (68.1, 13.6)
- moved R8 48.1 mm to (13.7, 44.7), turned to 180 degrees
- moved J6 47.0 mm to (12.2, 62.9), turned to 0 degrees
- moved R7 45.2 mm to (9.90, 44.7)
- moved J5 38.2 mm to (5.08, 16.4), turned to -90 degrees
- moved R4 34.9 mm to (56.8, 16.3), turned to 90 degrees
- moved Q1 34.0 mm to (25.0, 21.5), turned to 180 degrees
- moved U4 33.1 mm to (40.5, 43.9), turned to -90 degrees
- moved R9 27.1 mm to (23.8, 11.7)
- moved J1 21.5 mm to (47.0, 62.9)
- moved JP1 21.5 mm to (28.1, 16.4), turned to 180 degrees
- moved R5 18.2 mm to (53.2, 16.2)
- moved Q2 15.7 mm to (39.8, 21.8)
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Connections:
- A1 pad 10: unconnected-(A1-Pad10) -> GND_2_EN
- A1 pad 11: unconnected-(A1-Pad11) -> SCK
- A1 pad 12: unconnected-(A1-Pad12) -> MOSI
- A1 pad 13: unconnected-(A1-Pad13) -> MISO
- A1 pad 14: unconnected-(A1-Pad14) -> RX
- A1 pad 15: unconnected-(A1-Pad15) -> TX
- A1 pad 16: unconnected-(A1-Pad16) -> GND
- A1 pad 17: unconnected-(A1-Pad17) -> SDA
- A1 pad 18: unconnected-(A1-Pad18) -> SCL
- A1 pad 19: unconnected-(A1-Pad19) -> ONEWIRE
- A1 pad 2: unconnected-(A1-Pad2) -> +3V3
- A1 pad 20: unconnected-(A1-Pad20) -> LORA_CS
- A1 pad 21: unconnected-(A1-Pad21) -> LORA_RST
- A1 pad 22: unconnected-(A1-Pad22) -> SD_CS
- A1 pad 23: unconnected-(A1-Pad23) -> RX2
- A1 pad 24: unconnected-(A1-Pad24) -> TX2
- A1 pad 25: unconnected-(A1-Pad25) -> RTC_INT
- A1 pad 26: unconnected-(A1-Pad26) -> VBUS
- A1 pad 27: unconnected-(A1-Pad27) -> EN
- A1 pad 28: unconnected-(A1-Pad28) -> VBAT
- A1 pad 4: unconnected-(A1-Pad4) -> GND
- A1 pad 5: unconnected-(A1-Pad5) -> BUT_A
- A1 pad 6: unconnected-(A1-Pad6) -> SAT_EN
- A1 pad 7: unconnected-(A1-Pad7) -> GPS_RST
- A1 pad 8: unconnected-(A1-Pad8) -> WRITE_EN
- A1 pad 9: unconnected-(A1-Pad9) -> GND_1_EN
- AE1 pad 2: unconnected-(AE1-Pad2) -> Net-(U1-Pad9)
- J1 pad 1: unconnected-(J1-Pad1) -> +3V3
- J1 pad 2: unconnected-(J1-Pad2) -> ONEWIRE
- J1 pad 3: unconnected-(J1-Pad3) -> GND
- J2 pad 2: unconnected-(J2-Pad2) -> EN
- J5 pad 2: Net-(J5-Pad2) -> SD_CS
- J5 pad 3: WRITE_EN -> MOSI
- J6 pad 1: unconnected-(J6-Pad1) -> VBUS
- J6 pad 2: SD_CS -> GND
- J7 pad 1: unconnected-(J7-Pad1) -> GND_2
- J7 pad 2: unconnected-(J7-Pad2) -> +3V3
- J7 pad 3: unconnected-(J7-Pad3) -> RX
- J7 pad 4: unconnected-(J7-Pad4) -> TX
- JP1 pad 2: GND_2 -> GND_1
- JP2 pad 2: GND_1 -> GND_2
- Q1 pad 1: GND_2_EN -> GND_1_EN
- Q1 pad 2: GND_2 -> GND_1
- Q2 pad 1: GND_1_EN -> GND_2_EN
- Q2 pad 2: GND_1 -> GND_2
- R1 pad 2: SDA -> ONEWIRE
- R10 pad 1: Net-(C1-Pad1) -> Net-(J8-Pad2)
- R10 pad 2: +3V3 -> GND
- R2 pad 2: SDA -> ONEWIRE
- R3 pad 2: SCL -> SDA
- R4 pad 2: SCL -> SDA
- R5 pad 1: BUT_A -> +3V3
- R5 pad 2: +3V3 -> SCL
- R6 pad 2: BUT_A -> SCL
- R7 pad 1: Net-(J5-Pad2) -> BUT_A
- R7 pad 2: GND -> +3V3
- R8 pad 1: GND_2_EN -> +3V3
- R8 pad 2: GND -> BUT_A
- R9 pad 1: GND_1_EN -> Net-(J8-Pad2)
- U1 pad 1: unconnected-(U1-Pad1) -> GND
- U1 pad 10: unconnected-(U1-Pad10) -> GND
- U1 pad 13: unconnected-(U1-Pad13) -> +3V3
- U1 pad 2: unconnected-(U1-Pad2) -> MISO
- U1 pad 3: unconnected-(U1-Pad3) -> MOSI
- U1 pad 4: unconnected-(U1-Pad4) -> SCK
- U1 pad 5: unconnected-(U1-Pad5) -> LORA_CS
- U1 pad 6: unconnected-(U1-Pad6) -> LORA_RST
- U1 pad 8: unconnected-(U1-Pad8) -> GND
- U1 pad 9: unconnected-(U1-Pad9) -> Net-(U1-Pad9)
- U3 pad 10: unconnected-(U3-Pad10) -> GND_1
- U3 pad 3: unconnected-(U3-Pad3) -> +3V3
- U3 pad 7: unconnected-(U3-Pad7) -> GPS_RST
- U3 pad 8: unconnected-(U3-Pad8) -> SDA
- U3 pad 9: unconnected-(U3-Pad9) -> SCL
- U4 pad 1: Net-(U4-Pad1) -> +3V3
- U4 pad 2: Net-(U4-Pad2) -> GND
- U4 pad 3: Net-(BT1-Pad1) -> SCL
- U4 pad 4: GND -> SDA
- U4 pad 5: SDA -> unconnected-(U4-Pad5)
- U4 pad 6: SCL -> unconnected-(U4-Pad6)
- U4 pad 8: Net-(C1-Pad1) -> unconnected-(U4-Pad8)
Other:
- outline, holes or cut-outs redrawn
- board text added: "1 (GND)"
- board text added: "3V"
- board text added: "9 (ANT)"
- board text added: "D5"
- board text added: "GND"
- board text added: "GND_1"
- board text added: "RTC_INT"
- board text added: "RX"
- board text added: "SCL"
- board text added: "SDA"
- board text added: "TX"
- board text added: "VBUS"

Commit message: laid out power
Parts:
- moved J3 20.5 mm to (68.1, 34.1)
- moved JP1 3.26 mm to (25.7, 18.6), turned to 0 degrees
- moved JP2 2.61 mm to (40.5, 18.5)
- moved J4 1.90 mm to (68.1, 29.6), turned to 180 degrees
- moved R5 1.31 mm to (53.4, 17.5)
- moved R6 1.31 mm to (53.4, 21.3)
- moved R3 1.29 mm to (56.7, 21.4)
- moved R4 1.29 mm to (56.7, 17.6)
- moved Q1 1.03 mm to (25.5, 22.4)
- moved R12 0.94 mm to (29.4, 22.4)
- moved Q2 0.92 mm to (40.5, 22.4)
- moved R11 0.78 mm to (44.3, 22.4)
- moved R10 0.71 mm to (27.5, 12.4)
- moved R9 0.71 mm to (23.7, 12.4)
- moved R1 0.63 mm to (40.4, 12.4)
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Connections:
- AE1 pad 1: unconnected-(AE1-Pad1) -> GND
- J3 pad 2: unconnected-(J3-Pad2) -> RX2
- J3 pad 3: unconnected-(J3-Pad3) -> TX2
- J3 pad 4: unconnected-(J3-Pad4) -> +3V3
- J3 pad 6: unconnected-(J3-Pad6) -> GND
- J4 pad 1: unconnected-(J4-Pad1) -> GND
- J4 pad 6: unconnected-(J4-Pad6) -> SAT_EN
- J4 pad 7: unconnected-(J4-Pad7) -> VBAT
- J4 pad 8: unconnected-(J4-Pad8) -> GND
Routing:
- net GND: track 0.00 -> 344.1 mm, vias 0 -> 34
- net +3V3: track 0.00 -> 236.5 mm, vias 0 -> 22
- net GND_1: track 0.00 -> 118.6 mm, vias 0 -> 11
- net GND_2: track 0.00 -> 101.4 mm, vias 0 -> 11
- net VBUS: track 0.00 -> 94.5 mm, vias 0 -> 5
- net VBAT: track 0.00 -> 50.4 mm, vias 0 -> 3
Other:
- outline, holes or cut-outs redrawn
- board text added: "A1"
- board text added: "D11"
- board text added: "D12"
- board text added: "VBAT"

Commit message: fully routed
Routing:
- net SCL: track 0.00 -> 121.3 mm, vias 0 -> 8
- net SDA: track 0.00 -> 107.9 mm, vias 0 -> 7
- net MISO: track 0.00 -> 90.9 mm, vias 0 -> 8
- net SCK: track 0.00 -> 80.8 mm, vias 0 -> 4
- net MOSI: track 0.00 -> 69.0 mm, vias 0 -> 4
- net ONEWIRE: track 0.00 -> 68.6 mm, vias 0 -> 3
- net RTC_INT: track 0.00 -> 68.1 mm, vias 0 -> 5
- net LORA_RST: track 0.00 -> 67.1 mm, vias 0 -> 4
- net TX2: track 0.00 -> 65.1 mm, vias 0 -> 3
- net RX2: track 0.00 -> 65.1 mm, vias 0 -> 3
- net SD_CS: track 0.00 -> 61.5 mm, vias 0 -> 6
- net GPS_RST: track 0.00 -> 59.5 mm, vias 0 -> 4
- net LORA_CS: track 0.00 -> 54.9 mm, vias 0 -> 4
- net SAT_EN: track 0.00 -> 54.1 mm, vias 0 -> 3
- net RX: track 0.00 -> 49.7 mm, vias 0 -> 2
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Other:
- board text added: "OFF"
- board text added: "ON"
- board text added: "sweet-p"
- board text added: "v0.1"
- board text added: "write"
