File: ver_0.3/sweet-p.kicad_pcb (KiCad board)
At the start: 2 copper layers, 70 x 70 mm, 38 parts, among them J1 Screw_Terminal_01x03, J2 Conn_01x03_Female, J3 Conn_01x08_Female, J4 Conn_01x06_Female, J5 Micro_SD_Card, J6 Screw_Terminal_01x02, J7 Screw_Terminal_01x04, J8 Conn_01x03_Female, Q1 Q_NMOS_GDS, Q2 Q_NMOS_GDS, SW1 SW_Push, U1 adafruit_tpl511x, U2 RFM95W-868S2, U3 ssd1306, U4 Adafruit-Mini-GPS, U5 ds3231

Commit message: update
Parts:
- removed H4: MountingHole, MountingHole:MountingHole_3.2mm_M3
- removed J8: Conn_01x03_Female, Connector_PinSocket_2.54mm:PinSocket_1x03_P2.54mm_Vertical
- removed JP1, JP2: SolderJumper_2_Open, Jumper:SolderJumper-2_P1.3mm_Open_Pad1.0x1.5mm
- removed Q1, Q2: Q_NMOS_GDS, Package_TO_SOT_SMD:SOT-23
- removed the R10 at (27.5, 12.4)
- removed the R13 at (43.6, 42.7)
- removed the R9 at (23.7, 12.4)
- removed SW1: SW_Push, Button_Switch_THT:SW_Tactile_SPST_Angled_PTS645Vx31-2LFS
- added BZ1: PS1240P02BT, digikey-footprints:Piezo_Transducer_THT_PS1240P02BT, F.Cu at (96.3, 29.4)
- added D1: LED, LED_THT:LED_D5.0mm, F.Cu at (105.8, 31.9)
- added R15: 330, Resistor_THT:R_Axial_DIN0204_L3.6mm_D1.6mm_P7.62mm_Horizontal, F.Cu at (90.8, 40.5)
- added R16: 330, Resistor_SMD:R_0603_1608Metric_Pad0.98x0.95mm_HandSolder, F.Cu at (91.5, 45.9)
- added R17: 10K, Resistor_SMD:R_0603_1608Metric_Pad0.98x0.95mm_HandSolder, F.Cu at (51.4, 40.0)
- added R18: R, Resistor_THT:R_Axial_DIN0204_L3.6mm_D1.6mm_P7.62mm_Horizontal, F.Cu at (47.7, 39.9)
- added R3: 4.7K, Resistor_THT:R_Axial_DIN0204_L3.6mm_D1.6mm_P7.62mm_Horizontal, F.Cu at (104.8, 26.5)
- added R4: 4.7K, Resistor_SMD:R_0603_1608Metric_Pad0.98x0.95mm_HandSolder, F.Cu at (97.4, 43.4)
- added R8: 4.7K, Resistor_THT:R_Axial_DIN0204_L3.6mm_D1.6mm_P7.62mm_Horizontal, F.Cu at (22.7, 16.1)
- added S1: EG1218, digikey-footprints:Switch_Slide_11.6x4mm_EG1218, F.Cu at (37.9, 58.4)
- added S2: EG1218, digikey-footprints:Switch_Slide_11.6x4mm_EG1218, F.Cu at (1.45, 36.0)
- added U1: adafruit_ads1115, footprints:adafruit_ads1115, F.Cu at (95.5, 51.9)
- J2: value Conn_01x03_Female -> Conn_01x08_Female; footprint Connector_PinSocket_2.54mm:PinSocket_1x03_P2.54mm_Vertical -> Connector_PinSocket_2.54mm:PinSocket_1x08_P2.54mm_Vertical
- R10: renamed from R4; footprint Resistor_SMD:R_0603_1608Metric_Pad0.98x0.95mm_HandSolder -> Resistor_THT:R_Axial_DIN0204_L3.6mm_D1.6mm_P7.62mm_Horizontal
- R11: value R -> 4.7K; footprint Resistor_SMD:R_0603_1608Metric_Pad0.98x0.95mm_HandSolder -> Resistor_THT:R_Axial_DIN0204_L3.6mm_D1.6mm_P7.62mm_Horizontal
- R12, R14: value R -> 4.7K
- R6: renamed from R7; value 1K -> 4.7K
- R7: renamed from R8; value 10K -> 4.7K; footprint Resistor_THT:R_Axial_DIN0204_L3.6mm_D1.6mm_P7.62mm_Horizontal -> Resistor_SMD:R_0603_1608Metric_Pad0.98x0.95mm_HandSolder
- R9: renamed from R3; footprint Resistor_THT:R_Axial_DIN0204_L3.6mm_D1.6mm_P7.62mm_Horizontal -> Resistor_SMD:R_0603_1608Metric_Pad0.98x0.95mm_HandSolder
- moved R12 65.5 mm to (91.5, 43.4), turned to 0 degrees
- moved R13 55.4 mm to (18.5, 60.5), turned to 180 degrees
- moved R10 51.6 mm to (22.4, 56.2), turned to 180 degrees
- moved R9 51.6 mm to (18.6, 56.2), turned to 180 degrees
- moved R11 49.5 mm to (86.2, 48.9), turned to 0 degrees
- moved J2 44.1 mm to (87.0, 27.2), turned to 0 degrees
- moved R6 42.8 mm to (41.5, 15.8)
- moved R14 36.0 mm to (14.7, 60.5), turned to 0 degrees
- moved R7 31.3 mm to (26.5, 16.1)
- moved U2 17.9 mm to (60.0, 58.3), turned to -90 degrees
- moved J1 17.3 mm to (31.5, 70.5)
- moved J6 17.3 mm to (9.22, 70.5)
- moved J3 10.3 mm to (4.50, 56.1), turned to -90 degrees
- moved R5 9.79 mm to (45.3, 15.8), turned to 180 degrees
- moved H1 6.50 mm to (68.8, 72.7)
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- renumbered J6 to J3, J3 to J4, J4 to J5, J7 to J6, J5 to J7, R5 to R13, R6 to R5, U1 to U2, U2 to U4, U4 to U5, U5 to U6
Connections:
- A1 pad 10: GND_2_EN -> BUZZER
- A1 pad 25: RTC_INT -> LED
- A1 pad 26: VBUS -> DRIVE
- A1 pad 28: VBAT -> unconnected-(A1-Pad28)
- A1 pad 5: BUT_A -> A0
- A1 pad 8: WRITE_EN -> DONE
- A1 pad 9: GND_1_EN -> RTC_INT
- J2 pad 1: unconnected-(J2-Pad1) -> +3V3
- J2 pad 2: EN -> GND
- J2 pad 3: GND -> A0
- J3 pad 1: VBUS -> VEXT
- J4 pad 7: VBAT -> VEXT
- J6 pad 1: GND_2 -> GND
- R10 pad 1: +3V3 -> Net-(R10-Pad1)
- R10 pad 2: SDA -> GND
- R11 pad 1: GND_2_EN -> SAT_EN
- R12 pad 1: GND_1_EN -> SAT_EN
- R13 pad 1: +3V3 -> GND
- R13 pad 2: SCL -> Net-(R13-Pad2)
- R14 pad 1: +3V3 -> Net-(R13-Pad2)
- R14 pad 2: RTC_INT -> GND
- R5 pad 2: SCL -> SDA
- R6 pad 1: BUT_A -> +3V3
- R6 pad 2: +3V3 -> SDA
- R7 pad 2: BUT_A -> SCL
- R9 pad 1: +3V3 -> Net-(R10-Pad1)
- R9 pad 2: SDA -> GND
- U2 pad 1: unconnected-(U1-Pad1) -> Net-(S2-Pad1)
- U2 pad 2: unconnected-(U1-Pad2) -> GND
- U2 pad 3: unconnected-(U1-Pad3) -> Net-(S1-Pad2)
- U2 pad 4: unconnected-(U1-Pad4) -> DRIVE
- U2 pad 5: unconnected-(U1-Pad5) -> DRIVE
Other:
- board size 70 x 70 mm -> 73.5 x 76.2 mm
- board text removed: "write"

Commit message: update
Parts:
- removed the J2 at (87.0, 27.2)
- added J1: Conn_01x11_Female, Connector_PinSocket_2.54mm:PinSocket_1x11_P2.54mm_Vertical, F.Cu at (-10.1, 26.6)
- added R10: 100K, Resistor_SMD:R_0603_1608Metric_Pad0.98x0.95mm_HandSolder, F.Cu at (32.0, 37.8)
- added R11: 100K, Resistor_THT:R_Axial_DIN0204_L3.6mm_D1.6mm_P7.62mm_Horizontal, F.Cu at (28.9, 41.5)
- added R12: 100K, Resistor_SMD:R_0603_1608Metric_Pad0.98x0.95mm_HandSolder, F.Cu at (28.9, 37.8)
- added R9: 100K, Resistor_THT:R_Axial_DIN0204_L3.6mm_D1.6mm_P7.62mm_Horizontal, F.Cu at (32.1, 41.6)
- U6: moved to F.Cu
- moved D1 111.4 mm to (-2.12, 59.3)
- moved R19 97.5 mm to (-6.59, 34.7)
- moved R16 95.2 mm to (-2.95, 30.9)
- moved R20 95.0 mm to (-2.84, 34.6)
- moved R15 94.4 mm to (-6.55, 30.9)
- moved BZ1 84.2 mm to (14.2, 10.7)
- moved U1 74.3 mm to (21.2, 50.6), turned to 90 degrees
- moved R3 57.9 mm to (47.7, 36.1)
- moved R4 46.6 mm to (51.4, 36.0)
- moved U6 32.5 mm to (62.1, 13.6), turned to 90 degrees
- moved S2 29.8 mm to (-9.10, 63.9)
- moved A1 18.1 mm to (-2.60, 22.3)
- moved U3 16.8 mm to (8.31, 26.8)
- moved J3 15.7 mm to (-1.65, 70.5), turned to 0 degrees
- moved U4 13.5 mm to (11.1, 43.6)
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- renumbered J1 to J2, R9 to R13, R10 to R14, R11 to R15, R12 to R16, R13 to R17, R14 to R18, R15 to R19, R16 to R20, R17 to R21, R18 to R22
Connections:
- U1 pad 1: unconnected-(U1-Pad1) -> +3V3
- U1 pad 10: unconnected-(U1-Pad10) -> ADS_1
- U1 pad 11: unconnected-(U1-Pad11) -> Net-(U1-Pad11)
- U1 pad 2: unconnected-(U1-Pad2) -> GND
- U1 pad 3: unconnected-(U1-Pad3) -> SCL
- U1 pad 4: unconnected-(U1-Pad4) -> SDA
- U1 pad 8: unconnected-(U1-Pad8) -> ADS_3
- U1 pad 9: unconnected-(U1-Pad9) -> ADS_2
Other:
- board size 73.5 x 76.2 mm -> 84.3 x 76.2 mm
- board text removed: "1 (GND)"
- board text removed: "9 (ANT)"
- board text removed: "GND_1"
- board text removed: "RTC_INT"

Commit message: good layout -- need to check resistor locations
Parts:
- moved J1 38.5 mm to (6.03, 61.6), turned to 90 degrees
- moved R21 25.3 mm to (54.2, 14.9), turned to 90 degrees
- moved R22 22.3 mm to (54.2, 18.6), turned to 90 degrees
- moved R4 21.2 mm to (50.3, 14.9), turned to 90 degrees
- moved R3 17.7 mm to (50.4, 18.6), turned to 90 degrees
- moved R17 15.9 mm to (8.44, 55.3)
- moved R18 15.9 mm to (4.64, 55.3)
- moved R13 0.81 mm to (23.0, 55.3)
- moved R14 0.81 mm to (26.8, 55.3)
- moved S1 0.72 mm to (41.0, 55.7)

Commit message: fleshed out the power train
Parts:
- added C1: 0.1uF, Capacitor_THT:CP_Radial_Tantal_D4.5mm_P2.50mm, F.Cu at (2.07, 56.8)
- added C2: 0.1uF, Capacitor_THT:CP_Radial_Tantal_D4.5mm_P2.50mm, F.Cu at (7.80, 56.9)
- added C3: 10uF, Capacitor_THT:CP_Radial_Tantal_D4.5mm_P2.50mm, F.Cu at (13.5, 56.7)
- added JP1: Jumper_2_Open, Connector_PinHeader_2.54mm:PinHeader_1x02_P2.54mm_Vertical, F.Cu at (43.4, 55.1)
- added JP2: SolderJumper_2_Open, Jumper:SolderJumper-2_P1.3mm_Open_Pad1.0x1.5mm, F.Cu at (49.9, 65.5)
- added U2: MCP1700-3302E_TO, digikey-footprints:TO-92-3, F.Cu at (19.2, 57.1)
- moved R3 21.5 mm to (29.9, 55.8)
- moved R4 21.5 mm to (26.1, 55.8)
- moved R1 7.71 mm to (30.1, 52.2)
- moved R2 7.71 mm to (33.9, 52.2)
- moved A1 4.70 mm to (2.10, 22.1)
- moved S1 3.67 mm to (37.4, 54.8), turned to -90 degrees
- moved U7 2.93 mm to (65.0, 13.1)
- moved R20 2.76 mm to (-5.39, 35.7)
- moved R17 2.76 mm to (-9.10, 31.9)
- moved R19 2.76 mm to (-9.14, 35.8)
- moved R18 2.76 mm to (-5.50, 31.9)
- moved D1 2.21 mm to (-4.29, 58.9)
- moved R7 2.06 mm to (52.5, 18.4)
- moved R8 2.06 mm to (52.4, 14.7)
- moved R21 2.06 mm to (56.3, 14.7)
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- renumbered J3 to J1, J1 to J2, J2 to J3, R13 to R1, R6 to R10, R7 to R11, R8 to R12, R9 to R13, R10 to R14, R11 to R15, R12 to R16, R15 to R17, R16 to R18, R14 to R2, R17 to R3, R18 to R4, R1 to R5, R2 to R6, R3 to R7, R4 to R8, R5 to R9, U2 to U1, U1 to U3, U3 to U4, U4 to U5, U5 to U6, U6 to U7
Connections:
- A1 pad 26: DRIVE -> unconnected-(A1-Pad26)
- S2 pad 1: Net-(S2-Pad1) -> Net-(U2-Pad2)
- U1 pad 1: Net-(S2-Pad1) -> Net-(U1-Pad1)
- U1 pad 4: DRIVE -> +3V3
- U1 pad 5: DRIVE -> DONE

Commit message: fixed breakout
Parts:
- J2: value Conn_01x11_Female -> Conn_01x12_Female; footprint Connector_PinSocket_2.54mm:PinSocket_1x11_P2.54mm_Vertical -> Connector_PinSocket_2.54mm:PinSocket_2x06_P2.54mm_Vertical
- moved J2 35.4 mm to (-5.05, 28.0), turned to 0 degrees
- moved R19 17.6 mm to (7.90, 31.2)
- moved R20 17.6 mm to (11.7, 31.1)
- moved U2 14.9 mm to (4.62, 60.5), turned to 90 degrees
- moved R17 13.3 mm to (0.65, 41.0), turned to 90 degrees
- moved R18 8.25 mm to (0.60, 37.5), turned to 90 degrees
- moved R4 8.13 mm to (32.7, 60.6), turned to 90 degrees
- moved C2 7.04 mm to (14.3, 59.6)
- moved C1 7.04 mm to (8.57, 59.5)
- moved C3 7.04 mm to (20.0, 59.4)
- moved R2 6.55 mm to (27.4, 52.9), turned to -90 degrees
- moved R1 5.25 mm to (27.4, 56.7), turned to -90 degrees
- moved R3 2.94 mm to (32.7, 56.8), turned to -90 degrees
Connections:
- U6 pad 1: GND_1 -> GND

Commit message: update
Parts:
- removed J2: Conn_01x12_Female, Connector_PinSocket_2.54mm:PinSocket_2x06_P2.54mm_Vertical
- moved R1 11.2 mm to (38.5, 55.8), turned to 0 degrees
- moved JP1 10.6 mm to (53.9, 54.3), turned to 90 degrees
- moved R4 9.52 mm to (42.2, 60.5), turned to 180 degrees
- moved R18 9.00 mm to (-7.65, 33.9)
- moved R17 9.00 mm to (-7.60, 37.5)
- moved R2 7.86 mm to (34.7, 55.8), turned to 0 degrees
- moved S1 7.21 mm to (30.2, 55.4)
- moved R3 6.79 mm to (38.4, 60.5), turned to 0 degrees
- moved JP2 5.24 mm to (55.0, 64.3), turned to 180 degrees
- moved D1 1.45 mm to (-3.50, 60.1)
- moved S2 1.05 mm to (-9.60, 64.8)
- moved C3 0.80 mm to (20.8, 59.4)
- moved U2 0.80 mm to (5.42, 60.5)
- moved C1 0.80 mm to (9.37, 59.5)
- moved C2 0.80 mm to (15.1, 59.6)
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Connections:
- U6 pad 10: GND_1 -> GND

Commit message: update
Parts:
- added J2: Conn_01x03_Female, Connector_PinSocket_2.54mm:PinSocket_1x03_P2.54mm_Vertical, F.Cu at (55.1, 54.4)
- added J5: Conn_01x03_Female, Connector_PinSocket_2.54mm:PinSocket_1x03_P2.54mm_Vertical, F.Cu at (27.5, 36.8)
- moved JP1 14.7 mm to (56.3, 68.8), turned to -90 degrees
- moved R14 11.1 mm to (29.6, 48.6), turned to 0 degrees
- moved R13 9.47 mm to (25.8, 48.7), turned to 0 degrees
- moved R15 4.20 mm to (32.9, 42.8)
- moved R16 4.20 mm to (32.9, 39.1)
- moved U2 1.40 mm to (4.03, 60.5)
- moved D1 1.39 mm to (-4.88, 59.9)
- moved C1 1.33 mm to (8.05, 59.4)
- moved C2 1.28 mm to (13.8, 59.3)
- moved C3 1.14 mm to (19.6, 59.2)
- moved S1 0.50 mm to (29.7, 55.4)
- renumbered J5 to J6, J6 to J7, J7 to J8

Commit message: update
Parts:
- moved R19 54.6 mm to (58.8, 51.2), turned to 180 degrees
- moved R11 52.3 mm to (74.4, 37.1)
- moved R12 52.2 mm to (70.5, 37.0)
- moved C2 50.7 mm to (59.4, 81.6), turned to 90 degrees
- moved C1 50.7 mm to (53.6, 81.6), turned to 90 degrees
- moved R9 48.5 mm to (78.1, 32.5)
- moved R10 48.4 mm to (74.3, 32.4)
- moved R20 47.8 mm to (55.0, 51.2), turned to 180 degrees
- moved R17 47.4 mm to (33.6, 60.9)
- moved R18 47.4 mm to (33.6, 57.3)
- moved R5 47.0 mm to (70.5, 28.4)
- moved R6 47.0 mm to (74.3, 28.3)
- moved AE1 45.5 mm to (37.8, 69.3)
- moved U5 45.0 mm to (51.1, 64.1)
- moved J5 45.0 mm to (67.7, 56.9)
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Other:
- board size 84.3 x 76.2 mm -> 85 x 77 mm
- board text added: "11"
- board text added: "12"
- board text added: "VEX"
- board text added: "ads1115"
- board text added: "tpl5110"
- board text added: "v0.3"
- board text removed: "D11"
- board text removed: "D12"
- board text removed: "VBAT"
- board text removed: "v0.2"
