File: ver_0.3/sweet-p.kicad_pcb (KiCad board)
At the start: 2 copper layers, 85 x 77 mm, 51 parts, among them J1 Screw_Terminal_01x02, J2 Conn_01x03_Female, J3 Screw_Terminal_01x03, J4 Conn_01x08_Female, J5 Conn_01x03_Female, J6 Conn_01x06_Female, J7 Screw_Terminal_01x04, J8 Micro_SD_Card, U1 adafruit_tpl511x, U2 MCP1700-3302E_TO, U3 adafruit_ads1115, U4 ssd1306, U5 RFM95W-868S2, U6 Adafruit-Mini-GPS, U7 ds3231

Commit message: update
Parts:
- moved R19 22.3 mm to (36.6, 53.6), turned to -90 degrees
- moved R20 19.4 mm to (36.6, 57.4), turned to -90 degrees
- moved BZ1 6.45 mm to (58.2, 33.2), turned to -90 degrees
- moved R11 1.98 mm to (72.4, 37.1)
- moved R12 1.98 mm to (68.5, 37.1)
- moved R5 1.98 mm to (68.5, 28.4)
- moved R10 1.98 mm to (72.3, 32.5)
- moved R6 1.98 mm to (72.4, 28.4)
- moved R9 1.98 mm to (76.2, 32.5)
- moved JP2 1.60 mm to (92.9, 85.6)
- moved S1 1.28 mm to (67.8, 76.8)
- moved R16 1.01 mm to (68.8, 47.0)
- moved R15 1.01 mm to (65.2, 47.0)
- moved S2 0.88 mm to (28.1, 85.8)
- moved R18 0.72 mm to (32.9, 57.6)
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Other:
- board text added: "T1"
- board text added: "T2"
- board text added: "edgecollective.io/sweet-p"

Commit message: update
Parts:
- added JP3: Jumper_2_Open, Connector_PinHeader_2.54mm:PinHeader_1x02_P2.54mm_Vertical, F.Cu at (104.2, 81.8)
- added JP4: SolderJumper_2_Open, Jumper:SolderJumper-2_P1.3mm_Open_Pad1.0x1.5mm, F.Cu at (55.3, 83.3)
- added JP5: SolderJumper_2_Open, Jumper:SolderJumper-2_P1.3mm_Open_Pad1.0x1.5mm, F.Cu at (46.0, 83.3)
- JP1: value Jumper_2_Open -> SolderJumper_2_Open; footprint Connector_PinHeader_2.54mm:PinHeader_1x02_P2.54mm_Vertical -> Jumper:SolderJumper-2_P1.3mm_Open_Pad1.0x1.5mm
- moved JP1 5.10 mm to (89.5, 87.4), turned to 0 degrees
- moved JP2 4.42 mm to (96.9, 87.5), turned to 0 degrees
- moved C1 1.91 mm to (53.3, 79.7)
- moved C3 1.91 mm to (47.4, 79.7)
- moved C2 1.91 mm to (59.1, 79.7)
- moved U2 1.57 mm to (41.6, 77.6)
- moved S1 0.39 mm to (68.0, 76.5)
- moved D1 0.28 mm to (33.9, 80.8)
Connections:
- A1 pad 26: unconnected-(A1-Pad26) -> VUSB
- JP1 pad 1: Net-(C2-Pad1) -> VUSB
- JP1 pad 2: +3V3 -> Net-(U1-Pad4)
- JP2 pad 1: Net-(C2-Pad1) -> Net-(U1-Pad4)
- U1 pad 4: +3V3 -> Net-(U1-Pad4)
Other:
- board text added: "(3.3V)"
- board text added: "(usb)"

Commit message: update
Parts:
- moved R12 8.80 mm to (77.3, 36.8), turned to 180 degrees
- moved R5 8.75 mm to (77.3, 28.6), turned to 180 degrees
- moved R10 1.32 mm to (73.5, 32.9), turned to 180 degrees
- moved R9 1.25 mm to (77.4, 32.9)
- moved R6 1.15 mm to (73.5, 28.6), turned to 180 degrees
- moved R11 1.10 mm to (73.5, 36.8)
Routing:
- net GND: track 0.00 -> 380.0 mm, vias 0 -> 29
- net +3V3: track 0.00 -> 259.8 mm, vias 0 -> 19
- net VUSB: track 0.00 -> 70.3 mm, vias 0 -> 3
- net DONE: track 0.00 -> 4.56 mm

Commit message: update
Parts:
- added J1: Conn_01x02_Female, Connector_JST:JST_PH_B2B-PH-K_1x02_P2.00mm_Vertical, F.Cu at (39.9, 81.9)
- added J4: Conn_01x04_Female, Connector_PinSocket_2.54mm:PinSocket_1x04_P2.54mm_Vertical, F.Cu at (61.7, 76.2)
- JP1, JP2, JP4, JP5: moved to B.Cu
- moved JP4 14.1 mm to (42.2, 78.0), turned to 0 degrees
- moved C3 6.18 mm to (52.1, 83.7)
- moved U2 6.13 mm to (46.7, 81.0)
- moved C1 5.85 mm to (57.6, 83.7)
- moved C2 5.55 mm to (63.0, 83.7)
- moved JP5 5.43 mm to (46.8, 78.0), turned to 180 degrees
- moved D1 2.90 mm to (32.7, 78.1)
- moved S1 2.47 mm to (70.5, 76.9)
- moved R3 1.18 mm to (77.8, 81.3)
- moved R4 1.18 mm to (81.6, 81.3)
- moved R1 1.18 mm to (77.9, 76.6)
- moved R2 1.18 mm to (74.1, 76.6)
- turned JP1 to 180 degrees
- turned JP2 to 180 degrees
- renumbered J8 to J10, J1 to J2, J2 to J3, J3 to J5, J4 to J6, J5 to J7, J6 to J8, J7 to J9
Routing:
- net GND: track 380.0 -> 299.4 mm, vias 29 -> 24
- net +3V3: track 259.8 -> 225.3 mm, vias 19 -> 16
- net VUSB: track 70.3 -> 64.8 mm
Other:
- board text added: "VEXT"
- board text removed: "VBUS"

Commit message: continuing routing
Parts:
- moved C2 5.46 mm to (57.5, 83.7)
- moved C1 5.35 mm to (62.9, 83.7)
- moved JP1 0.65 mm to (89.5, 88.0), turned to -90 degrees
- moved D1 0.57 mm to (32.9, 78.7)
- moved JP2 0.53 mm to (96.8, 88.1), turned to 90 degrees
Routing:
- net GND: track 299.4 -> 382.5 mm, vias 24 -> 28
- net Net-(C2-Pad1): track 0.00 -> 82.8 mm, vias 0 -> 8
- net VUSB: track 64.8 -> 6.17 mm, vias 3 -> 2
- net +3V3: track 225.3 -> 264.2 mm, vias 16 -> 19
- net VEXT: track 0.00 -> 23.0 mm, vias 0 -> 1
- net Net-(R3-Pad2): track 0.00 -> 16.0 mm
- net Net-(U1-Pad4): track 0.00 -> 15.8 mm, vias 0 -> 2

Commit message: nearly all routed
Parts:
- moved R8 52.2 mm to (40.0, 24.7), turned to 180 degrees
- moved R7 49.7 mm to (43.7, 24.6), turned to 180 degrees
- moved R19 8.02 mm to (32.4, 60.4), turned to 90 degrees
- moved S2 5.31 mm to (27.9, 80.5), turned to -90 degrees
- moved R20 4.29 mm to (32.4, 56.5), turned to 90 degrees
- moved R17 2.42 mm to (35.2, 60.4)
- moved R18 2.42 mm to (35.2, 56.8)
- moved D1 2.36 mm to (35.1, 78.0), turned to 180 degrees
Connections:
- A1 pad 5: A0 -> unconnected-(A1-Pad5)
- U6 pad 12: unconnected-(U6-Pad12) -> +3V3
Routing:
- net SCL: track 0.02 -> 196.5 mm, vias 0 -> 12
- net SDA: track 0.00 -> 188.6 mm, vias 0 -> 10
- net VEXT: track 23.0 -> 155.5 mm, vias 1 -> 7
- net SAT_EN: track 0.00 -> 115.1 mm, vias 0 -> 4
- net DONE: track 4.56 -> 114.5 mm, vias 0 -> 5
- net RX: track 0.00 -> 93.9 mm, vias 0 -> 4
- net VUSB: track 6.17 -> 99.7 mm, vias 2 -> 4
- net TX: track 0.00 -> 91.7 mm, vias 0 -> 6
- net RX2: track 0.00 -> 83.1 mm, vias 0 -> 3
- net TX2: track 0.00 -> 81.1 mm, vias 0 -> 1
- net ONEWIRE: track 0.00 -> 74.0 mm, vias 0 -> 2
- net Net-(D1-Pad2): track 0.00 -> 68.7 mm, vias 0 -> 4
- net RTC_INT: track 0.00 -> 65.3 mm, vias 0 -> 4
- net SCK: track 0.00 -> 61.4 mm, vias 0 -> 7
- net Net-(C1-Pad1): track 0.00 -> 53.7 mm, vias 0 -> 7
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
Commit message: final layout and gerbers
Parts:
- J3: value Conn_01x03_Female -> Conn_01x04_Female; footprint Connector_PinSocket_2.54mm:PinSocket_1x03_P2.54mm_Vertical -> Connector_PinSocket_2.54mm:PinSocket_1x04_P2.54mm_Vertical
- moved J3 2.55 mm to (95.3, 76.2)
Connections:
- A1 pad 27: EN -> unconnected-(A1-Pad27)
- J3 pad 1: Net-(J3-Pad1) -> GND
- J3 pad 2: +3V3 -> Net-(S1-Pad2)
- J3 pad 3: DONE -> +3V3
- S1 pad 2: Net-(J3-Pad1) -> Net-(S1-Pad2)
- U1 pad 3: Net-(J3-Pad1) -> Net-(S1-Pad2)
Routing:
- net GPS_RST: track 0.00 -> 73.2 mm, vias 0 -> 6
- net LORA_RST: track 0.00 -> 52.7 mm, vias 0 -> 3
- net +3V3: track 269.3 -> 309.3 mm, vias 20 -> 21
- net Net-(S1-Pad2): track 0.00 -> 27.8 mm, vias 0 -> 1
- net Net-(J3-Pad1): track 27.8 -> 0.00 mm, vias 1 -> 0
- net MOSI: track 44.3 -> 71.0 mm, vias 1 -> 4
- net MISO: track 52.5 -> 79.0 mm, vias 2 -> 4
- net GND: track 369.6 -> 394.9 mm, vias 27 -> 28
- net Net-(C2-Pad1): track 82.7 -> 83.6 mm, vias 7 -> 6
- net SDA: vias 10 -> 9
- net SCL: vias 12 -> 11
Other:
- board text added: "2(MISO)"
- board text added: "9(ANT)"
- board text added: "ADS_1"
- board text added: "ADS_2"
- board text added: "ADS_3"
- board text added: "DELAY"
- board text added: "DONE"
- board text added: "DRIVE"
- board text added: "VDD"
