File: ver_0.3/sweet-p.kicad_sch (KiCad schematic)
At the start: 41 parts, among them J1 Screw_Terminal_01x03, J2 Conn_01x03_Female, J3 Conn_01x08_Female, J4 Conn_01x06_Female, J5 Micro_SD_Card, J6 Screw_Terminal_01x02, J7 Screw_Terminal_01x04, J8 Conn_01x03_Female, Q1 Q_NMOS_GDS, Q2 Q_NMOS_GDS, SW1 SW_Push, U1 adafruit_tpl511x, U2 RFM95W-868S2, U3 ssd1306, U4 Adafruit-Mini-GPS, U5 ds3231

Commit message: update
Parts:
- removed H4: MountingHole, MountingHole:MountingHole_3.2mm_M3, symbol Mechanical:MountingHole
- removed J2, J8: Conn_01x03_Female, Connector_PinSocket_2.54mm:PinSocket_1x03_P2.54mm_Vertical, symbol Connector:Conn_01x03_Female
- removed JP1, JP2: SolderJumper_2_Open, Jumper:SolderJumper-2_P1.3mm_Open_Pad1.0x1.5mm, symbol Jumper:SolderJumper_2_Open
- removed Q1, Q2: Q_NMOS_GDS, Package_TO_SOT_SMD:SOT-23, symbol Device:Q_NMOS_GDS
- removed R10: 10K, Resistor_SMD:R_0603_1608Metric_Pad0.98x0.95mm_HandSolder, symbol Device:R
- removed R7: 1K, Resistor_SMD:R_0603_1608Metric_Pad0.98x0.95mm_HandSolder, symbol Device:R
- removed R8: 10K, Resistor_THT:R_Axial_DIN0204_L3.6mm_D1.6mm_P7.62mm_Horizontal, symbol Device:R
- removed SW1: SW_Push, Button_Switch_THT:SW_Tactile_SPST_Angled_PTS645Vx31-2LFS, symbol Switch:SW_Push
- added BZ1: PS1240P02BT, digikey-footprints:Piezo_Transducer_THT_PS1240P02BT, symbol dk_Alarms-Buzzers-and-Sirens:PS1240P02BT
- added D1: LED, LED_THT:LED_D5.0mm, symbol Device:LED
- added J2: Conn_01x08_Female, Connector_PinSocket_2.54mm:PinSocket_1x08_P2.54mm_Vertical, symbol Connector:Conn_01x08_Female
- added R14, R3: 4.7K, Resistor_THT:R_Axial_DIN0204_L3.6mm_D1.6mm_P7.62mm_Horizontal, symbol Device:R
- added R15: 330, Resistor_THT:R_Axial_DIN0204_L3.6mm_D1.6mm_P7.62mm_Horizontal, symbol Device:R
- added R16: 330, Resistor_SMD:R_0603_1608Metric_Pad0.98x0.95mm_HandSolder, symbol Device:R
- added R4: 4.7K, Resistor_SMD:R_0603_1608Metric_Pad0.98x0.95mm_HandSolder, symbol Device:R
- added S2: EG1218, digikey-footprints:Switch_Slide_11.6x4mm_EG1218, symbol dk_Slide-Switches:EG1218
- added U1: adafruit_ads1115, footprints:adafruit_ads1115, symbol sweet-p:adafruit_ads1115
- R11: value R -> 4.7K; footprint Resistor_SMD:R_0603_1608Metric_Pad0.98x0.95mm_HandSolder -> Resistor_THT:R_Axial_DIN0204_L3.6mm_D1.6mm_P7.62mm_Horizontal
- R12: value R -> 4.7K
- R13: renamed from R?; footprint Resistor_THT:R_Axial_DIN0204_L3.6mm_D1.6mm_P7.62mm_Horizontal -> Resistor_SMD:R_0603_1608Metric_Pad0.98x0.95mm_HandSolder
- R9: value 10K -> 4.7K; footprint Resistor_THT:R_Axial_DIN0204_L3.6mm_D1.6mm_P7.62mm_Horizontal -> Resistor_SMD:R_0603_1608Metric_Pad0.98x0.95mm_HandSolder
- gave numbers to parts that had none: 1
- renumbered J6 to J3, J3 to J4, J4 to J5, J7 to J6, J5 to J7, R13 to R17, R14 to R18, R3 to R5, R4 to R6, R5 to R7, R6 to R8, U1 to U2, U2 to U4, U4 to U5, U5 to U6
Connections:
- net GND_2 is gone; now on net GND: J6.1 (Pin_1)
- net +3V3: now also J2.1 (Pin_1)
- net GND: now also U2.2 (GND), BZ1.2, D1.1 (K), J2.2 (Pin_2), R14.2, R15.2, R16.2
- net GPS_RST: now also J2.5 (Pin_5)
- net RTC_INT: now also A1.9 (A4), J2.7 (Pin_7); no longer A1.25 (D13)
- net SAT_EN: now also R11.1, R12.1, J2.4 (Pin_4)
- net at R13.2, S1.3: now also R14.1
- net at R10.1, S1.1: now also R9.1
- net at U2.1 (VDD): now also S2.1
- net DRIVE: now reaches U2.4 (DRIVE)
- net DRIVE: now also A1.26 (USB), U2.5 (DONE)
- net BUT_A renamed A0
- net A0: now also J2.3 (Pin_3)
- removed net GND_1_EN: A1.9 (A4), R12.1
- net GND_2_EN renamed BUZZER
- net BUZZER: now also BZ1.1, J2.8 (Pin_8); no longer R11.1
- net VBAT: no longer names the net of A1.28 (VBAT)
- net VBAT: no longer J4.7 (Pin_7)
- net VBUS renamed VEXT
- net VEXT: now also J4.7 (Pin_7), S2.2; no longer A1.26 (USB)
- net WRITE_EN renamed DONE
- net DONE: now also J2.6 (Pin_6), R15.1, R16.1
- new net: D1.2 (A), R3.2, R4.2
- new net LED: A1.25 (D13), R3.1, R4.1
Other:
- note added: "breakout"
- note added: "buzzer"
- note added: "depth_sensor"
- note added: "ext display"
- note added: "external LED"
- note added: "gps"
- note added: "lora"
- note added: "onewire"
- note added: "pull-downs"
- note added: "rtc"
- note removed: "could be used for 1-wire or for serial"
- note removed: "write permit"
- moved on the sheet: AE1, J1, J3, J6, R1, R2, R5, R6, R7, R8, U4

Commit message: update
Parts:
- removed J2: Conn_01x08_Female, Connector_PinSocket_2.54mm:PinSocket_1x08_P2.54mm_Vertical, symbol Connector:Conn_01x08_Female
- added J1: Conn_01x11_Female, Connector_PinSocket_2.54mm:PinSocket_1x11_P2.54mm_Vertical, symbol Connector:Conn_01x11_Female
- added R10, R12: 100K, Resistor_SMD:R_0603_1608Metric_Pad0.98x0.95mm_HandSolder, symbol Device:R
- added R11, R9: 100K, Resistor_THT:R_Axial_DIN0204_L3.6mm_D1.6mm_P7.62mm_Horizontal, symbol Device:R
- renumbered J1 to J2, R9 to R13, R10 to R14, R11 to R15, R12 to R16, R13 to R17, R14 to R18, R15 to R19, R16 to R20, R17 to R21, R18 to R22
Connections:
- net +3V3: now also U1.1 (VIN), J1.1 (Pin_1)
- net A0: now also J1.3 (Pin_3)
- net BUZZER: now also J1.8 (Pin_8)
- net DONE: now also J1.6 (Pin_6)
- net GND: now also U1.2 (GND), J1.2 (Pin_2), R11.2, R12.2
- net GPS_RST: now also J1.5 (Pin_5)
- net RTC_INT: now also J1.7 (Pin_7)
- net SAT_EN: now also J1.4 (Pin_4)
- net SCL: now also U1.3 (SCL)
- net SDA: now also U1.4 (SDA)
- net VEXT: now also R10.1, R9.1
- net ADS_1: now reaches U1.10 (A1)
- net ADS_1: now also J1.9 (Pin_9)
- net at U1.11 (A0): now also R10.2, R11.1, R12.1, R9.2
- net ADS_3: now reaches U1.8 (A3)
- net ADS_3: now also J1.11 (Pin_11)
- net ADS_2: now reaches U1.9 (A2)
- net ADS_2: now also J1.10 (Pin_10)
Other:
- note added: "vext measure"
- moved on the sheet: U1

Commit message: fleshed out the power train
Parts:
- added C1, C2: 0.1uF, Capacitor_THT:CP_Radial_Tantal_D4.5mm_P2.50mm, symbol Device:C_Polarized
- added C3: 10uF, Capacitor_THT:CP_Radial_Tantal_D4.5mm_P2.50mm, symbol Device:C_Polarized
- added JP1: Jumper_2_Open, Connector_PinHeader_2.54mm:PinHeader_1x02_P2.54mm_Vertical, symbol Jumper:Jumper_2_Open
- added JP2: SolderJumper_2_Open, Jumper:SolderJumper-2_P1.3mm_Open_Pad1.0x1.5mm, symbol Jumper:SolderJumper_2_Open
- added U2: MCP1700-3302E_TO, digikey-footprints:TO-92-3, symbol dk_PMIC-Voltage-Regulators-Linear:MCP1700-3302E_TO
- renumbered J3 to J1, J1 to J2, J2 to J3, R13 to R1, R6 to R10, R7 to R11, R8 to R12, R9 to R13, R10 to R14, R11 to R15, R12 to R16, R15 to R17, R16 to R18, R14 to R2, R17 to R3, R18 to R4, R1 to R5, R2 to R6, R3 to R7, R4 to R8, R5 to R9, U2 to U1, U1 to U3, U3 to U4, U4 to U5, U5 to U6, U6 to U7
Connections:
- net +3V3: now also U1.4 (DRIVE), JP1.2 (B), JP2.2 (B)
- net DONE: now also U1.5 (DONE)
- net GND: now also U6.1 (GND), C1.2, C2.2, C3.2, U2.1 (GND)
- net GND_1: no longer U6.1 (GND)
- net at U1.1 (VDD): now also C2.1, C3.1, JP1.1 (A), JP2.1 (A), U2.3 (VOUT); no longer S2.1
- removed net DRIVE: A1.26 (USB), U1.4 (DRIVE), U1.5 (DONE)
- new net: C1.1, S2.1, U2.2 (VIN)
Other:
- note added: "3.3V LDO"
- note added: "<--- 5V max, 450 mA capable when using sat modem"
- note added: "low power timer"
- moved on the sheet: H1, H2, H3, J1, R1, R2, R3, R4, S1, S2, U1

Commit message: fixed breakout
Parts:
- removed J2: Conn_01x11_Female, Connector_PinSocket_2.54mm:PinSocket_1x11_P2.54mm_Vertical, symbol Connector:Conn_01x11_Female
- added J2: Conn_01x12_Female, Connector_PinSocket_2.54mm:PinSocket_2x06_P2.54mm_Vertical, symbol Connector:Conn_01x12_Female
Connections:
- net +3V3: now also J2.1 (Pin_1)
- net A0: now also J2.3 (Pin_3)
- net ADS_1: now also J2.9 (Pin_9)
- net ADS_2: now also J2.10 (Pin_10)
- net ADS_3: now also J2.11 (Pin_11)
- net BUZZER: now also J2.8 (Pin_8)
- net DONE: now also J2.6 (Pin_6)
- net GND: now also J2.2 (Pin_2)
- net GPS_RST: now also J2.5 (Pin_5)
- net RTC_INT: now also J2.7 (Pin_7)
- net SAT_EN: now also J2.4 (Pin_4)
- net VEXT: now also J2.12 (Pin_12)

Commit message: update
Parts:
- removed J2: Conn_01x12_Female, Connector_PinSocket_2.54mm:PinSocket_2x06_P2.54mm_Vertical, symbol Connector:Conn_01x12_Female
Connections:
- net GND_1 is gone; now on net GND: U6.10 (GND)
Other:
- note removed: "breakout"
Changed lines of the file:
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@@
+    (stroke (width 0) (type default) (color 0 0 0 0))
+  )
+  (wire (pts (xy -132.08 138.43) (xy -125.095 138.43))
     (stroke (width 0) (type default) (color 0 0 0 0))
   )
@@
     (stroke (width 0) (type default) (color 0 0 0 0))
   )
-  (wire (pts (xy -55.88 -74.295) (xy -44.45 -74.295))
-    (stroke (width 0) (type default) (color 0 0 0 0))
-  )
   (wire (pts (xy -143.51 -124.46) (xy -123.825 -124.46))
     (stroke (width 0) (type default) (color 0 0 0 0))
@@
     (effects (font (size 5 5)) (justify left bottom))
   )
-  (text "breakout" (at -60.96 -85.725 0)
-    (effects (font (size 5 5)) (justify left bottom))
-  )
   (text "ssd1306" (at 33.02 100.33 0)
     (effects (font (size 1.27 1.27)) (justify left bottom))
@@
     )
   )
-  (global_label "VEXT" (shape input) (at -44.45 -48.895 180) (fields_autoplaced)
-    (effects (font (size 1.27 1.27)) (justify right))
-    (property "Intersheet References" "${INTERSHEET_REFS}" (id 0) (at -51.2779 -48.9744 0)
-      (effects (font (size 1.27 1.27)) (justify right) hide)
-    )
-  )
   (global_label "SAT_EN" (shape input) (at -261.62 30.48 0) (fields_autoplaced)
     (effects (font (size 1.27 1.27)) (justify left))
@@
     )
   )
-  (global_label "GND_1" (shape input) (at -132.08 138.43 0) (fields_autoplaced)
-    (effects (font (size 1.27 1.27)) (justify left))
-    (property "Intersheet References" "${INTERSHEET_REFS}" (id 0) (at -123.6193 138.3506 0)
-      (effects (font (size 1.27 1.27)) (justify left) hide)
-    )
-  )
   (global_label "SCL" (shape input) (at 45.72 114.3 0) (fields_autoplaced)
     (effects (font (size 1.27 1.27)) (justify left))
@@
     )
   )
-  (global_label "ADS_2" (shape input) (at -44.45 -53.975 180) (fields_autoplaced)
-    (effects (font (size 1.27 1.27)) (justify right))
-    (property "Intersheet References" "${INTERSHEET_REFS}" (id 0) (at -52.6083 -53.8956 0)
-      (effects (font (size 1.27 1.27)) (justify right) hide)
-    )
-  )
   (global_label "VEXT" (shape input) (at -58.42 3.81 90) (fields_autoplaced)
     (effects (font (size 1.27 1.27)) (justify left))
@@
     )
   )
-  (global_label "A0" (shape input) (at -44.45 -71.755 180) (fields_autoplaced)
-    (effects (font (size 1.27 1.27)) (justify right))
-    (property "Intersheet References" "${INTERSHEET_REFS}" (id 0) (at -49.1612 -71.6756 0)
-      (effects (font (size 1.27 1.27)) (justify right) hide)
-    )
-  )
   (global_label "RTC_INT" (shape input) (at 77.47 180.34 0) (fields_autoplaced)
     (effects (font (size 1.27 1.27)) (justify left))
@@
     )
   )
-  (global_label "ADS_1" (shape input) (at -44.45 -56.515 180) (fields_autoplaced)
-    (effects (font (size 1.27 1.27)) (justify right))
-    (property "Intersheet References" "${INTERSHEET_REFS}" (id 0) (at -52.6083 -56.4356 0)
-      (effects (font (size 1.27 1.27)) (justify right) hide)
-    )
-  )
   (global_label "DONE" (shape input) (at -77.47 -124.46 0) (fields_autoplaced)
     (effects (font (size 1.27 1.27)) (justify left))
@@
     )
   )
-  (global_label "GPS_RST" (shape input) (at -44.45 -66.675 180) (fields_autoplaced)
-    (effects (font (size 1.27 1.27)) (justify right))
-    (property "Intersheet References" "${INTERSHEET_REFS}" (id 0) (at -55.0274 -66.5956 0)
-      (effects (font (size 1.27 1.27)) (justify right) hide)
-    )
-  )
   (global_label "ADS_2" (shape input) (at -88.265 8.255 0) (fields_autoplaced)
     (effects (font (size 1.27 1.27)) (justify left))
@@
     )
   )
-  (global_label "DONE" (shape input) (at -44.45 -64.135 180) (fields_autoplaced)
-    (effects (font (size 1.27 1.27)) (justify right))
-    (property "Intersheet References" "${INTERSHEET_REFS}" (id 0) (at -51.9431 -64.0556 0)
-      (effects (font (size 1.27 1.27)) (justify right) hide)
-    )
-  )
   (global_label "RX" (shape input) (at -59.69 76.2 180) (fields_autoplaced)
     (effects (font (size 1.27 1.27)) (justify right))
@@
     )
   )
-  (global_label "ADS_3" (shape input) (at -44.45 -51.435 180) (fields_autoplaced)
-    (effects (font (size 1.27 1.27)) (justify right))
-    (property "Intersheet References" "${INTERSHEET_REFS}" (id 0) (at -52.6083 -51.3556 0)
-      (effects (font (size 1.27 1.27)) (justify right) hide)
-    )
-  )
   (global_label "SDA" (shape input) (at 45.72 118.11 0) (fields_autoplaced)
     (effects (font (size 1.27 1.27)) (justify left))
@@
     )
   )
-  (global_label "BUZZER" (shape input) (at -44.45 -59.055 180) (fields_autoplaced)
-    (effects (font (size 1.27 1.27)) (justify right))
-    (property "Intersheet References" "${INTERSHEET_REFS}" (id 0) (at -54.3017 -58.9756 0)
-      (effects (font (size 1.27 1.27)) (justify right) hide)
-    )
-  )
   (global_label "SDA" (shape input) (at 44.45 187.96 180) (fields_autoplaced)
     (effects (font (size 1.27 1.27)) (justify right))
     (property "Intersheet References" "${INTERSHEET_REFS}" (id 0) (at 38.4688 187.8806 0)
-      (effects (font (size 1.27 1.27)) (justify right) hide)
-    )
-  )
-  (global_label "RTC_INT" (shape input) (at -44.45 -61.595 180) (fields_autoplaced)
-    (effects (font (size 1.27 1.27)) (justify right))
-    (property "Intersheet References" "${INTERSHEET_REFS}" (id 0) (at -54.2412 -61.5156 0)
-      (effects (font (size 1.27 1.27)) (justify right) hide)
-    )
-  )
-  (global_label "SAT_EN" (shape input) (at -44.45 -69.215 180) (fields_autoplaced)
-    (effects (font (size 1.27 1.27)) (justify right))
-    (property "Intersheet References" "${INTERSHEET_REFS}" (id 0) (at -53.576 -69.1356 0)
       (effects (font (size 1.27 1.27)) (justify right) hide)
     )
@@
     (pin "1")
   )
-  (symbol (lib_id "power:+3V3") (at -44.45 -76.835 0) (unit 1)
-    (in_bom yes) (on_board yes) (fields_autoplaced)
-    (property "Reference" "#PWR07" (id 0) (at -44.45 -73.025 0)
-      (effects (font (size 1.27 1.27)) hide)
-    )
-    (property "Value" "+3V3" (id 1) (at -44.45 -81.915 0))
-    (property "Footprint" "" (id 2) (at -44.45 -76.835 0)
-      (effects (font (size 1.27 1.27)) hide)
-    )
-    (property "Datasheet" "" (id 3) (at -44.45 -76.835 0)
-      (effects (font (size 1.27 1.27)) hide)
-    )
-    (pin "1")
-  )
   (symbol (lib_id "sweet-p:adafruit_tpl511x") (at -86.36 -133.35 0) (unit 1)
     (in_bom yes) (on_board yes) (fields_autoplaced)
@@
     (pin "1")
   )
-  (symbol (lib_id "power:GND") (at -55.88 -74.295 0) (unit 1)
-    (in_bom yes) (on_board yes)
-    (property "Reference" "#PWR08" (id 0) (at -55.88 -67.945 0)
-      (effects (font (size 1.27 1.27)) hide)
-    )
-    (property "Value" "GND" (id 1) (at -62.23 -73.025 0)
-      (effects (font (size 1.27 1.27)) (justify left))
-    )
-    (property "Footprint" "" (id 2) (at -55.88 -74.295 0)
-      (effects (font (size 1.27 1.27)) hide)
-    )
-    (property "Datasheet" "" (id 3) (at -55.88 -74.295 0)
+  (symbol (lib_id "power:GND") (at -125.095 138.43 0) (unit 1)
+    (in_bom yes) (on_board yes) (fields_autoplaced)
+    (property "Reference" "#PWR?" (id 0) (at -125.095 144.78 0)
+      (effects (font (size 1.27 1.27)) hide)
+    )
+    (property "Value" "GND" (id 1) (at -125.095 143.51 0))
+    (property "Footprint" "" (id 2) (at -125.095 138.43 0)
+      (effects (font (size 1.27 1.27)) hide)
+    )
+    (property "Datasheet" "" (id 3) (at -125.095 138.43 0)
       (effects (font (size 1.27 1.27)) hide)
     )
@@
     (pin "1")
   )
-  (symbol (lib_id "Connector:Conn_01x12_Female") (at -39.37 -64.135 0) (unit 1)
-    (in_bom yes) (on_board yes) (fields_autoplaced)
-    (property "Reference" "J2" (id 0) (at -36.83 -64.1351 0)
-      (effects (font (size 1.27 1.27)) (justify left))
-    )
-    (property "Value" "Conn_01x12_Female" (id 1) (at -36.83 -61.5951 0)
-      (effects (font (size 1.27 1.27)) (justify left))
-    )
-    (property "Footprint" "Connector_PinSocket_2.54mm:PinSocket_2x06_P2.54mm_Vertical" (id 2) (at -39.37 -64.135 0)
-      (effects (font (size 1.27 1.27)) hide)
-    )
-    (property "Datasheet" "~" (id 3) (at -39.37 -64.135 0)
-      (effects (font (size 1.27 1.27)) hide)
-    )
-    (pin "1")
-    (pin "10")
-    (pin "11")
-    (pin "12")
-    (pin "2")
-    (pin "3")
-    (pin "4")
-    (pin "5")
-    (pin "6")
-    (pin "7")
-    (pin "8")
-    (pin "9")
-  )
   (symbol (lib_id "Device:R") (at -125.73 -50.8 0) (unit 1)
     (in_bom yes) (on_board yes) (fields_autoplaced)
@@
       (reference "#PWR06") (unit 1) (value "GND") (footprint "")
     )
-    (path "/80b1e8b0-c14a-43f3-8c02-df696b45978a"
-      (reference "#PWR07") (unit 1) (value "+3V3") (footprint "")
-    )
-    (path "/cba62e84-41d5-4142-a06a-c47b4bef012c"
-      (reference "#PWR08") (unit 1) (value "GND") (footprint "")
-    )
     (path "/edd9ae1f-b214-4924-bbe9-6791b913da4c"
       (reference "#PWR09") (unit 1) (value "+3V3") (footprint "")
@@
       (reference "#PWR043") (unit 1) (value "GND") (footprint "")
     )
+    (path "/d7a87d32-960d-4b6c-9ec6-e9cc6793a0ff"
+      (reference "#PWR?") (unit 1) (value "GND") (footprint "")
+    )
     (path "/183fe64b-877b-44e3-91b5-dd0a6ba3e1e1"
       (reference "A1") (unit 1) (value "Adafruit_Feather_M0_Express") (footprint "Module:Adafruit_Feather")
@@
       (reference "J1") (unit 1) (value "Screw_Terminal_01x02") (footprint "TerminalBlock_Phoenix:TerminalBlock_Phoenix_PT-1,5-2-5.0-H_1x02_P5.00mm_Horizontal")
     )
-    (path "/f1f261cd-aaf9-4dd2-beec-91fdb571c969"
-      (reference "J2") (unit 1) (value "Conn_01x12_Female") (footprint "Connector_PinSocket_2.54mm:PinSocket_2x06_P2.54mm_Vertical")
-    )
     (path "/356a682b-39b5-417e-8373-9ae81bd97f29"

Commit message: update
Parts:
- added J2, J5: Conn_01x03_Female, Connector_PinSocket_2.54mm:PinSocket_1x03_P2.54mm_Vertical, symbol Connector:Conn_01x03_Female
- renumbered J5 to J6, J6 to J7, J7 to J8
Connections:
- net +3V3: now also J2.2 (Pin_2)
- net ADS_1: now also J5.1 (Pin_1)
- net ADS_2: now also J5.2 (Pin_2)
- net ADS_3: now also J5.3 (Pin_3)
- net DONE: now also J2.3 (Pin_3)
- net at S1.2, U1.3 (DELAY): now also J2.1 (Pin_1)

Commit message: update
Parts:
- removed H2: MountingHole, MountingHole:MountingHole_3.2mm_M3, symbol Mechanical:MountingHole
Changed lines of the file:
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@@
     (pin "2")
-  )
-  (symbol (lib_id "Mechanical:MountingHole") (at 228.6 -5.715 0) (unit 1)
-    (in_bom yes) (on_board yes) (fields_autoplaced)
-    (property "Reference" "H2" (id 0) (at 231.14 -6.9851 0)
-      (effects (font (size 1.27 1.27)) (justify left))
-    )
-    (property "Value" "MountingHole" (id 1) (at 231.14 -4.4451 0)
-      (effects (font (size 1.27 1.27)) (justify left))
-    )
-    (property "Footprint" "MountingHole:MountingHole_3.2mm_M3" (id 2) (at 228.6 -5.715 0)
-      (effects (font (size 1.27 1.27)) hide)
-    )
-    (property "Datasheet" "~" (id 3) (at 228.6 -5.715 0)
-      (effects (font (size 1.27 1.27)) hide)
-    )
   )
   (symbol (lib_id "power:GND") (at -135.89 -39.37 0) (unit 1)
@@
       (reference "H1") (unit 1) (value "MountingHole") (footprint "MountingHole:MountingHole_3.2mm_M3")
     )
-    (path "/c1b87c36-4435-4ea9-8dcd-3792ff53f4a3"
-      (reference "H2") (unit 1) (value "MountingHole") (footprint "MountingHole:MountingHole_3.2mm_M3")
-    )
     (path "/318e249e-412d-4076-86d9-3d57986e4360"

Commit message: update
Parts:
- added H?: MountingHole, MountingHole:MountingHole_3.2mm_M3, symbol Mechanical:MountingHole
Other:
- moved on the sheet: H1, H3
Changed lines of the file:
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@@
     (pin "1")
   )
-  (symbol (lib_id "Mechanical:MountingHole") (at 228.6 4.445 0) (unit 1)
-    (in_bom yes) (on_board yes) (fields_autoplaced)
-    (property "Reference" "H3" (id 0) (at 231.14 3.1749 0)
-      (effects (font (size 1.27 1.27)) (justify left))
-    )
-    (property "Value" "MountingHole" (id 1) (at 231.14 5.7149 0)
-      (effects (font (size 1.27 1.27)) (justify left))
-    )
-    (property "Footprint" "MountingHole:MountingHole_3.2mm_M3" (id 2) (at 228.6 4.445 0)
-      (effects (font (size 1.27 1.27)) hide)
-    )
-    (property "Datasheet" "~" (id 3) (at 228.6 4.445 0)
-      (effects (font (size 1.27 1.27)) hide)
-    )
-  )
-  (symbol (lib_id "Mechanical:MountingHole") (at 218.44 -15.875 0) (unit 1)
-    (in_bom yes) (on_board yes) (fields_autoplaced)
-    (property "Reference" "H1" (id 0) (at 220.98 -17.1451 0)
-      (effects (font (size 1.27 1.27)) (justify left))
-    )
-    (property "Value" "MountingHole" (id 1) (at 220.98 -14.6051 0)
-      (effects (font (size 1.27 1.27)) (justify left))
-    )
-    (property "Footprint" "MountingHole:MountingHole_3.2mm_M3" (id 2) (at 218.44 -15.875 0)
-      (effects (font (size 1.27 1.27)) hide)
-    )
-    (property "Datasheet" "~" (id 3) (at 218.44 -15.875 0)
+  (symbol (lib_id "Mechanical:MountingHole") (at -268.605 -81.28 0) (unit 1)
+    (in_bom yes) (on_board yes) (fields_autoplaced)
+    (property "Reference" "H3" (id 0) (at -266.065 -82.5501 0)
+      (effects (font (size 1.27 1.27)) (justify left))
+    )
+    (property "Value" "MountingHole" (id 1) (at -266.065 -80.0101 0)
+      (effects (font (size 1.27 1.27)) (justify left))
+    )
+    (property "Footprint" "MountingHole:MountingHole_3.2mm_M3" (id 2) (at -268.605 -81.28 0)
+      (effects (font (size 1.27 1.27)) hide)
+    )
+    (property "Datasheet" "~" (id 3) (at -268.605 -81.28 0)
+      (effects (font (size 1.27 1.27)) hide)
+    )
+  )
+  (symbol (lib_id "Mechanical:MountingHole") (at -278.765 -101.6 0) (unit 1)
+    (in_bom yes) (on_board yes) (fields_autoplaced)
+    (property "Reference" "H1" (id 0) (at -276.225 -102.8701 0)
+      (effects (font (size 1.27 1.27)) (justify left))
+    )
+    (property "Value" "MountingHole" (id 1) (at -276.225 -100.3301 0)
+      (effects (font (size 1.27 1.27)) (justify left))
+    )
+    (property "Footprint" "MountingHole:MountingHole_3.2mm_M3" (id 2) (at -278.765 -101.6 0)
+      (effects (font (size 1.27 1.27)) hide)
+    )
+    (property "Datasheet" "~" (id 3) (at -278.765 -101.6 0)
       (effects (font (size 1.27 1.27)) hide)
     )
@@
   )
   (symbol (lib_name "GND_2") (lib_id "power:GND") (at 198.12 24.13 180) (unit 1)
-    (in_bom yes) (on_board yes) (fields_autoplaced)
+    (in_bom yes) (on_board yes)
     (property "Reference" "#PWR017" (id 0) (at 198.12 17.78 0)
       (effects (font (size 1.27 1.27)) hide)
@@
     (pin "2")
   )
+  (symbol (lib_id "Mechanical:MountingHole") (at -273.05 -90.805 0) (unit 1)
+    (in_bom yes) (on_board yes) (fields_autoplaced)
+    (property "Reference" "H?" (id 0) (at -270.51 -92.0751 0)
+      (effects (font (size 1.27 1.27)) (justify left))
+    )
+    (property "Value" "MountingHole" (id 1) (at -270.51 -89.5351 0)
+      (effects (font (size 1.27 1.27)) (justify left))
+    )
+    (property "Footprint" "MountingHole:MountingHole_3.2mm_M3" (id 2) (at -273.05 -90.805 0)
+      (effects (font (size 1.27 1.27)) hide)
+    )
+    (property "Datasheet" "~" (id 3) (at -273.05 -90.805 0)
+      (effects (font (size 1.27 1.27)) hide)
+    )
+  )
   (symbol (lib_id "power:GND") (at 175.26 -135.89 0) (unit 1)
     (in_bom yes) (on_board yes) (fields_autoplaced)
@@
       (reference "H3") (unit 1) (value "MountingHole") (footprint "MountingHole:MountingHole_3.2mm_M3")
     )
+    (path "/7ebd7910-fb13-4782-93e2-0b357871bfda"
+      (reference "H?") (unit 1) (value "MountingHole") (footprint "MountingHole:MountingHole_3.2mm_M3")
+    )
     (path "/45c0a94b-fa0f-4fe7-8b75-e0ec592276a1"
