File: ver_0.3/sweet-p.kicad_sch (KiCad schematic)
At the start: 51 parts, among them J1 Screw_Terminal_01x02, J2 Conn_01x03_Female, J3 Screw_Terminal_01x03, J4 Conn_01x08_Female, J5 Conn_01x03_Female, J6 Conn_01x06_Female, J7 Screw_Terminal_01x04, J8 Micro_SD_Card, U1 adafruit_tpl511x, U2 MCP1700-3302E_TO, U3 adafruit_ads1115, U4 ssd1306, U5 RFM95W-868S2, U6 Adafruit-Mini-GPS, U7 ds3231

Commit message: update
Parts:
- added JP1, JP2, JP5: SolderJumper_2_Open, Jumper:SolderJumper-2_P1.3mm_Open_Pad1.0x1.5mm, symbol Jumper:SolderJumper_2_Open
- gave numbers to parts that had none: 1
- renumbered JP1 to JP3, JP2 to JP4
Connections:
- net +3V3: now also JP2.2 (B); no longer U1.4 (DRIVE)
- net at C2.1, C3.1, JP3.1 (A)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: now also JP5.2 (B)
- net at C1.1, S2.1, U2.2 (VIN): now also JP5.1 (A)
- net VUSB: now reaches A1.26 (USB)
- net VUSB: now also JP1.1 (A)
- new net: JP1.2 (B), JP2.1 (A), U1.4 (DRIVE)

Commit message: update
Parts:
- added J1: Conn_01x02_Female, Connector_JST:JST_PH_B2B-PH-K_1x02_P2.00mm_Vertical, symbol Connector:Conn_01x02_Female
- added J4: Conn_01x04_Female, Connector_PinSocket_2.54mm:PinSocket_1x04_P2.54mm_Vertical, symbol Connector:Conn_01x04_Female
- renumbered J8 to J10, J1 to J2, J2 to J3, J3 to J5, J4 to J6, J5 to J7, J6 to J8, J7 to J9
Connections:
- net +3V3: now also J4.2 (Pin_2)
- net GND: now also J1.2 (Pin_2), J4.1 (Pin_1)
- net SCL: now also J4.3 (Pin_3)
- net SDA: now also J4.4 (Pin_4)
- net VEXT: now also J1.1 (Pin_1)

Commit message: nearly all routed
Connections:
- net +3V3: now also U6.12 (VIN)
- net A0: no longer names the net of A1.5 (DAC0/A0)
- no-connect marks 0 -> 24
Changed lines of the file:
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@@
   (junction (at -123.825 -132.08) (diameter 0) (color 0 0 0 0)
   )
+  (junction (at -162.56 135.89) (diameter 0) (color 0 0 0 0)
+  )
   (junction (at -113.03 -155.575) (diameter 0) (color 0 0 0 0)
   )
@@
   (junction (at -193.675 -132.08) (diameter 0) (color 0 0 0 0)
   )
+  (no_connect (at -104.775 15.875))
+  (no_connect (at 186.69 53.34))
+  (no_connect (at 186.69 39.37))
+  (no_connect (at 186.69 34.29))
+  (no_connect (at -88.265 0.635))
+  (no_connect (at -88.265 19.685))
+  (no_connect (at -149.86 133.35))
+  (no_connect (at -149.86 140.97))
+  (no_connect (at -246.38 120.65))
+  (no_connect (at -153.67 13.97))
+  (no_connect (at -246.38 113.03))
+  (no_connect (at -168.91 3.81))
+  (no_connect (at -246.38 125.73))
+  (no_connect (at -149.86 143.51))
+  (no_connect (at -104.775 19.685))
+  (no_connect (at -153.67 24.13))
+  (no_connect (at -153.67 29.21))
+  (no_connect (at -246.38 123.19))
+  (no_connect (at -246.38 115.57))
+  (no_connect (at -246.38 118.11))
+  (no_connect (at 186.69 31.75))
+  (no_connect (at 186.69 63.5))
+  (no_connect (at -149.86 138.43))
+  (no_connect (at 186.69 36.83))
   (wire (pts (xy -77.47 71.12) (xy -59.69 71.12))
     (stroke (width 0) (type default) (color 0 0 0 0))
@@
     (stroke (width 0) (type default) (color 0 0 0 0))
   )
+  (wire (pts (xy -132.08 149.86) (xy -132.08 143.51))
+    (stroke (width 0) (type default) (color 0 0 0 0))
+  )
   (wire (pts (xy 74.93 180.34) (xy 77.47 180.34))
     (stroke (width 0) (type default) (color 0 0 0 0))
@@
     (stroke (width 0) (type default) (color 0 0 0 0))
   )
+  (wire (pts (xy -162.56 135.89) (xy -162.56 149.86))
+    (stroke (width 0) (type default) (color 0 0 0 0))
+  )
   (wire (pts (xy -107.315 -140.97) (xy -107.315 -132.08))
     (stroke (width 0) (type default) (color 0 0 0 0))
@@
   )
   (wire (pts (xy -111.125 -132.08) (xy -107.315 -132.08))
+    (stroke (width 0) (type default) (color 0 0 0 0))
+  )
+  (wire (pts (xy -162.56 149.86) (xy -132.08 149.86))
     (stroke (width 0) (type default) (color 0 0 0 0))
   )
@@
     )
   )
-  (global_label "A0" (shape input) (at -153.67 29.21 0) (fields_autoplaced)
-    (effects (font (size 1.27 1.27)) (justify left))
-    (property "Intersheet References" "${INTERSHEET_REFS}" (id 0) (at -148.9588 29.1306 0)
-      (effects (font (size 1.27 1.27)) (justify left) hide)
-    )
-  )

Commit message: final layout and gerbers
Parts:
- removed J3: Conn_01x03_Female, Connector_PinSocket_2.54mm:PinSocket_1x03_P2.54mm_Vertical, symbol Connector:Conn_01x03_Female
- added J3: Conn_01x04_Female, Connector_PinSocket_2.54mm:PinSocket_1x04_P2.54mm_Vertical, symbol Connector:Conn_01x04_Female
Connections:
- net +3V3: now also J3.3 (Pin_3)
- net DONE: now also J3.4 (Pin_4)
- net GND: now also J3.1 (Pin_1)
- net at S1.2, U1.3 (DELAY): now also J3.2 (Pin_2)
- net EN: no longer names the net of A1.27 (EN)
- no-connect marks 24 -> 25
