File: ver_0.4a/sweet-p.kicad_sch (KiCad schematic)
At the start: 41 parts, among them J1 Screw_Terminal_01x03, J10 Micro_SD_Card, J2 Screw_Terminal_01x02, J3 Conn_01x04_Female, J5 Screw_Terminal_01x05, J6 Conn_01x02_Socket, J7 Conn_01x06_Pin, J8 Conn_01x08_Socket, SW1 SW_Push, U1 adafruit_tpl511x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

Commit message: update
Parts:
- added C1, C3: 10uF, symbol Device:C
- added U2: MCP1700x-120xxTO, Package_TO_SOT_THT:TO-92_Inline, symbol Regulator_Linear:MCP1700x-120xxTO
Connections:
- net +3V3: now also C3.1, U2.3 (VO)
- net 5V_TIMER: now also C1.1, U2.2 (VI)
- new net: C1.2, C3.2, U2.1 (GND)
