File: ver_1/sweet-p.kicad_pcb (KiCad board)
At the start: 2 copper layers, 83 x 73 mm, 45 parts, among them J10 Conn_01x01_Socket, J11 Conn_01x03_Pin, J2 Screw_Terminal_01x02, J3 Conn_01x04_Female, J4 to '+' of converter, J5 Screw_Terminal_01x05, J6 Conn_01x02_Socket, J7 Conn_01x06_Pin, J8 Conn_01x08_Socket, J9 to '-' of probe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

Commit message: update
Parts:
- added H5: MountingHole, MountingHole:MountingHole_3.2mm_M3, F.Cu at (-101.6, 74.3)
- added H6: MountingHole, MountingHole:MountingHole_3.2mm_M3, F.Cu at (-86.6, 74.3)
- moved R4 230.2 mm to (-128.3, 31.7), turned to 0 degrees
- moved R3 227.3 mm to (-124.5, 31.7), turned to 0 degrees
- moved J7 215.0 mm to (-109.8, 13.2), turned to -90 degrees
- moved U2 207.4 mm to (-56.5, 71.8)
- moved J11 193.1 mm to (-97.0, 46.0)
- moved Q2 191.0 mm to (-113.3, 68.8)
- moved J9 190.3 mm to (-76.9, 92.7)
- moved J4 190.1 mm to (-112.3, 92.5)
- moved R2 190.0 mm to (-138.4, 57.1), turned to 90 degrees
- moved J6 187.7 mm to (-138.4, 45.1), turned to 180 degrees
- moved R11 187.4 mm to (-104.0, 58.8), turned to 90 degrees
- moved J3 187.0 mm to (-129.9, 46.0)
- moved R19 187.0 mm to (-115.2, 52.2)
- moved R20 187.0 mm to (-115.2, 48.3)
- moved U1 187.0 mm to (-124.7, 44.0)
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Other:
- board size 83 x 73 mm -> 103.5 x 89.5 mm
- board text added: "5VTimer"
- board text added: "Current to Voltage Converter"
- board text added: "sweet-p ver 1.0"
- board text removed: "5VT"
- board text removed: "DRIVE"
- board text removed: "converter"
- board text removed: "sweet-p ver 0.4a"

Commit message: ver 1 completed
Parts:
- removed J10: Conn_01x01_Socket, Connector_PinSocket_2.54mm:PinSocket_1x01_P2.54mm_Vertical
- added R5: 10K, Resistor_THT:R_Axial_DIN0204_L3.6mm_D1.6mm_P7.62mm_Horizontal, F.Cu at (96.8, 41.2)
- R1, R17, R18, R2: value 4.7K -> 10K
- R19, R20: value 330 -> 10K
- moved R11 237.3 mm to (132.9, 73.3), turned to 0 degrees
- moved R12 233.2 mm to (129.0, 73.3), turned to 0 degrees
- moved D1 231.3 mm to (159.1, 58.4), turned to 90 degrees
- moved R8 217.1 mm to (149.4, 57.0), turned to 0 degrees
- moved SW1 217.1 mm to (157.2, 46.5)
- moved R10 214.9 mm to (132.7, 68.0), turned to 0 degrees
- moved R9 211.3 mm to (128.9, 68.0), turned to 0 degrees
- moved J8 210.6 mm to (130.4, 84.5)
- moved R15 209.7 mm to (83.1, 54.0)
- moved R3 209.7 mm to (83.5, 58.8)
- moved R16 209.7 mm to (79.4, 54.0)
- moved R4 209.7 mm to (79.7, 58.8)
- moved R7 209.7 mm to (145.7, 57.0), turned to 0 degrees
- moved C2 208.7 mm to (81.5, 92.0), turned to 0 degrees
- moved J11 208.3 mm to (110.0, 69.2)
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Connections:
- net A5 renamed FORCE_A5
- J7 pad 5: RX -> Net-(J7-Pin_5)
- J9 pad 1: unconnected-(J9-Pin_1-Pad1) -> GND
Routing:
- net GND: track 0.00 -> 409.7 mm, vias 0 -> 21
- net +3V3: track 0.00 -> 294.4 mm, vias 0 -> 13
- net SDA: track 0.00 -> 156.0 mm, vias 0 -> 5
- net D12: track 0.00 -> 147.3 mm, vias 0 -> 3
- net SCL: track 0.00 -> 146.4 mm, vias 0 -> 6
- net 5V_TIMER: track 0.00 -> 129.9 mm, vias 0 -> 8
- net 5V_DC: track 0.00 -> 117.3 mm, vias 0 -> 6
- net VEXT: track 0.00 -> 115.9 mm, vias 0 -> 7
- net TX_A4: track 0.00 -> 113.9 mm, vias 0 -> 4
- net RX_D2: track 0.00 -> 96.6 mm, vias 0 -> 2
- net FORCE_A5: track 0.00 -> 95.1 mm, vias 0 -> 2
- net A0: track 0.00 -> 88.6 mm, vias 0 -> 3
- net A3: track 0.00 -> 83.2 mm, vias 0 -> 3
- net LED: track 0.00 -> 79.6 mm, vias 0 -> 2
- net BATT_A1: track 0.00 -> 61.6 mm, vias 0 -> 3
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Other:
- board size 103.5 x 89.5 mm -> 102.8 x 88.9 mm
- board text added: "5V_DC"
- board text added: "Converter Minus"
- board text added: "SAT_EN"
- board text added: "VEXT SWITCHED"
- board text added: "VIN"
- board text removed: "Probe Minus"
- board text removed: "SEN"
